File: revA/control.kicad_sch (KiCad schematic)
At the start: 112 parts, among them J1 JST 03B-SR, J2 JST 03B-SR, SW1 KMR231NG LFS, SW2 KMR231NG LFS, U14 MR25H10MDF, U15 ATSAMD51J20A-A, U16 DAC121S101Q, U17 MAX708RESA-T, U18 DAC121S101Q, U19 DAC121S101Q, Y1 12MHz

Commit message: working
Parts:
- removed BOM1, BOM2: JST 03SR Jumper, Resistor_SMD:R_0603_1608Metric, symbol SierraLobo:BOMTIE
- removed C2, C3: 6pF, Capacitor_SMD:C_0402_1005Metric, symbol Device:C
- removed C57, C58, C59: 0.1uF, Capacitor_SMD:C_0402_1005Metric, symbol Device:C
- removed D6, D7, D8: SK6805-EC3210R, payload-interface-board:SK6812-EC3210F-RA, symbol FP-Interface-Card:SK6812-EC321F_4
- removed J1, J2: JST 03B-SR, Connector_JST:JST_SH_SM03B-SRSS-TB_1x03-1MP_P1.00mm_Horizontal, symbol Connector_Generic:Conn_01x03
- removed R3, R4: 27, Capacitor_SMD:C_0402_1005Metric, symbol Device:R_US
- removed R80, R81: 100, Resistor_SMD:R_0603_1608Metric, symbol Device:R_US
- removed R88, R89, R90, R91: 1k, Resistor_SMD:R_0402_1005Metric, symbol Device:R_US
- removed Y1: 12MHz, symbol Device:Crystal
- added C66, C67: 8pF, Capacitor_SMD:C_0402_1005Metric, symbol Device:C
- added C68, C69, C70, C71, C72, C73, C74, C75: 0.1uF, Capacitor_SMD:C_0402_1005Metric, symbol Device:C
- added C76, C77, C78, C79, C82: 1uF, Capacitor_SMD:C_0603_1608Metric, symbol Device:C
- added C80, C81: 10uF, Capacitor_SMD:C_0805_2012Metric, symbol Device:C
- added C83, C9: 10uF, symbol Device:C
- added C9: 0.1uF, symbol Device:C
- added C9: 4.7uF, symbol Device:C
- added L2: 10uH, Inductor_SMD:L_1210_3225Metric, symbol Device:L
- added P2: FTSH-105-01-F-DV-K-TR, Connector_PinHeader_1.27mm:PinHeader_2x05_P1.27mm_Vertical_SMD, symbol Connector_Generic:Conn_02x05_Odd_Even
- added P3: TSM-105-01-F-SV, Connector_PinHeader_2.54mm:PinHeader_1x05_P2.54mm_Vertical_SMD_Pin1Right, symbol Connector_Generic:Conn_01x05
- added R44, R46: 1k, symbol Device:R_US
- added Y2: 32.768kHz, SierraLobo:Crystal_SMD_3215-2Pin_3.2x1.5mm, symbol Device:Crystal
- D?: renamed from D5; value SK6805-EC3210R -> SK6812MINI; footprint payload-interface-board:SK6812-EC3210F-RA -> LED_SMD:LED_SK6812MINI_PLCC4_3.5x3.5mm_P1.75mm; symbol FP-Interface-Card:SK6812-EC321F_4 -> LED:SK6812MINI
- R45: value 1k -> 10k
- R77: value 10k -> 1k; footprint Resistor_SMD:R_0402_1005Metric -> (none); now fitted
- R87: value 1k -> 499; footprint Resistor_SMD:R_0402_1005Metric -> (none)
Connections:
- net 3V3A is gone; now on net +3V3: C9.1
- net QSPI_SCLK is gone; now on net QSPI/SCK: U14.6 (SCK)
- net QSPI_SD0 is gone; now on net QSPI/DATA0: U14.5 (SI)
- net QSPI_SD1 is gone; now on net QSPI/DATA1: U14.2 (SO)
- net QSPI_SD2 is gone; now on net QSPI/DATA2: U14.3 (~{WP})
- net QSPI_SD3 is gone; now on net QSPI/DATA3: U14.7 (~{HOLD})
- net XOUT is gone; now on net SWCLK: R45.2
- net 3V3D: no longer C35.1, R42.2, R67.1, R69.1, R77.2, U14.8 (VDD), U17.2 (VCC)
- net GND: now also D?.2 (VSS), R69.2, U15.22 (GND), U15.33 (GND), U15.47 (GND), U15.54 (GND), U15.7 (GNDANA), C66.2, C67.2, C68.2, C69.2, C70.2, C71.2, C72.2, C73.2, C74.2, C75.2, C79.2, C80.2, C81.2, C82.1, C83.2, C9.2, C9.2, C9.2, P2.3 (Pin_3), P2.5 (Pin_5), P2.9 (Pin_9), P3.5 (Pin_5); no longer D?.1 (VSS)
- net LED_DIN: no longer R87.2
- net SWCLK: now also U15.57 (PA30), P2.4 (Pin_4)
- net USB_D+: now also U15.45 (PA24)
- net USB_D-: now also U15.46 (PA25)
- net WDT_WDI: now also R69.1, U15.44 (PA23)
- net XTAL1: now reaches U15.1 (PA00)
- net XTAL1: now also C66.1, Y2.1
- net AIN2: now reaches U15.11 (PB08)
- net AIN4: now reaches U15.13 (PA04)
- net AIN5: now reaches U15.14 (PA05)
- net AIN6: now reaches U15.15 (PA06)
- net AIN7: now reaches U15.16 (PA07)
- net QSPI/DATA0: now reaches U15.17 (PA08)
- net QSPI/DATA1: now reaches U15.18 (PA09)
- net QSPI/DATA2: now reaches U15.19 (PA10)
- net XTAL2: now reaches U15.2 (PA01)
- net XTAL2: now also C67.1, Y2.2
- net QSPI/DATA3: now reaches U15.20 (PA11)
- net QSPI/SCK: now reaches U15.23 (PB10)
- net QSPI/CS: now reaches U15.24 (PB11)
- net QSPI/CS: now also R42.1, U14.1 (~{CS})
- net AIN0: now reaches U15.3 (PA02)
- net TX: now reaches U15.37 (PA18)
- net TX: now also U15.39 (PB16)
- net at U15.38 (PA19): now also R44.1
- net +3V3: now reaches U15.4 (PA03)
- net +3V3: now also C35.1, R42.2, R45.1, R67.1, U14.8 (VDD), U15.8 (VDDANA), U17.2 (VCC), C68.1, C69.1, C70.1, C71.1, C72.1, C73.1, C74.1, C75.1, C76.1, C77.1, C78.1, C79.1, C80.1, C81.1, C9.1, C9.1, C9.1, P2.1 (Pin_1), P3.1 (Pin_1)
- net at U15.40 (PB17): now also R77.1
- net NEOPIXEL_DIN: now reaches U15.42 (PA21)
- net NEOPIXEL_DIN: now also R87.2
- net TX_DEBUG: now reaches U15.49 (PB22)
- net at U15.50 (PB23): now also R46.1
- net ~{RST}: now reaches U15.52 (~{RESET})
- net ~{RST}: now also C52.2, JP2.2 (B), R67.2, R86.1, P2.10 (Pin_10)
- net VDDCORE: now reaches U15.53 (VDDCORE)
- net VDDCORE: now also C82.2, C83.1, L2.2
- net VSW: now reaches U15.55 (VSW)
- net VSW: now also L2.1
- net SWDIO: now reaches U15.58 (PA31)
- net SWDIO: now also P2.2 (Pin_2)
- net AIN15: now reaches U15.64 (PB03)
- removed net QSPI_SS: R42.1, R43.2, U14.1 (~{CS})
- removed net ~{PICO_RST}: C52.2, JP2.2 (B), R67.2, R69.2, R86.1
- new net RX: R44.2, R77.2
- new net RX_DEBUG: R46.2
- no-connect marks 1 -> 4
Other:
- note added: "ANAREF"
- note added: "Crystal"
- note added: "DECOUPLING"
- note added: "Debug Serial Header"
- note added: "JTAG Port"
- note added: "SERCOM1/IOSET3"
- note added: "SERCOM5/IOSET1"
- note added: "STATUS LED"
- note added: "cut or DNI for flight"
- note removed: "12MHz Crystal"
- note removed: "Debug / Programming Port"
- note removed: "Make sure R3 and R4 are close to RP2040"
- note removed: "STATUS LEDs"
- note removed: "double check qspi po"
- moved on the sheet: C35, C52, C53, C54, C55, C56, C9, D?, JP1, JP2, R4, R42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

Commit message: exported init pdf
Parts:
- removed C10, C60, C62, C64, C76, C77, C78, C79, C8: 1uF, Capacitor_SMD:C_0603_1608Metric, symbol Device:C
- removed C11, C12, C13, C14, C15, C16 (x2), C6, C61, C63, C65, C68, C69, C7, C70, C71, C9: 0.1uF, Capacitor_SMD:C_0402_1005Metric, symbol Device:C
- removed C17: 10uF, Capacitor_SMD:C_0805_2012Metric, symbol Device:C
- removed C53, C54, C55: ?, symbol Device:C
- removed JP1: Wire Cut Jumper, Resistor_SMD:R_0603_1608Metric, symbol Jumper:Jumper_2_Bridged
- removed R100, R92, R96: 330, Resistor_SMD:R_0603_1608Metric, symbol Device:R_US
- removed R101, R102, R103, R4, R43, R93, R94, R95, R97, R98, R99: 1k, Resistor_SMD:R_0402_1005Metric, symbol Device:R_US
- removed R4 (x23): 0, Resistor_SMD:R_0603_1608Metric, symbol Device:R_US
- removed R4 (x4): 10k, Resistor_SMD:R_0402_1005Metric, symbol Device:R_US
- removed R73, R74: 100, Resistor_SMD:R_0603_1608Metric, symbol Device:R_US
- removed R83, R84, R85: ?, Resistor_SMD:R_0603_1608Metric, symbol Device:R_US
- removed SW1: KMR231NG LFS, SierraLobo:KMR2_4.6X2.8, symbol Switch:SW_SPST
- removed U16, U18, U19: DAC121S101Q, Package_TO_SOT_SMD:TSOT-23-6, symbol SierraLobo:DAC121S101Q
- J?: renamed from P3; value TSM-105-01-F-SV -> Conn_01x06; footprint Connector_PinHeader_2.54mm:PinHeader_1x05_P2.54mm_Vertical_SMD_Pin1Right -> Connector_PinHeader_2.54mm:PinHeader_1x06_P2.54mm_Vertical_SMD_Pin1Right; symbol Connector_Generic:Conn_01x05 -> Connector_Generic:Conn_01x06; Manufacturer Samtec -> (none); Mfr. Part No TSM-105-01-F-SV -> (none)
Connections:
- net +3V3: now also U15.21 (VDDIOB), U15.34 (VDDIO), U15.48 (VDDIO), U15.56 (VDDIO); no longer J?.1 (Pin_1)
- net GND: no longer J?.5 (Pin_5)
Other:
- note removed: "BOOTSEL"
- note removed: "DACs"
- note removed: "Make sure C10 is close to pin 44 of RP2040"
- note removed: "Make sure C8 is close to pin 45 of RP2040"
- note removed: "RP2040 MCU"
- note removed: "cut for flight"
- moved on the sheet: C35, C52, C56, C66, C67, C72, C73, C74, C75, C80, C81, D?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

Commit message: working
Parts:
- removed C9: 0.1uF, symbol Device:C
- removed C9: 4.7uF, symbol Device:C
- removed R44: 1k, symbol Device:R_US
- added C16: 0.1uF, Capacitor_SMD:C_0603_1608Metric, symbol Device:C
- added LED1: YELLOW, SierraLobo:APA2107x, symbol Device:D
- added LED4: RED, SierraLobo:APA2107x, symbol Device:D
- added Q2: PNP, symbol Simulation_SPICE:PNP
- added Q6: MMDT2222A, Package_TO_SOT_SMD:SOT-363_SC-70-6, symbol SierraLobo:MMDT2222
- added R104, R28: 1.5k, Resistor_SMD:R_0402_1005Metric, symbol Device:R_US
- added R18: 330k, Resistor_SMD:R_0603_1608Metric, symbol Device:R_US
- added R19: 110k, Resistor_SMD:R_0603_1608Metric, symbol Device:R_US
- added R22, R26, R27, R30, R31: 10k, Resistor_SMD:R_0603_1608Metric, symbol Device:R_US
- added R23: 100k, Resistor_SMD:R_0603_1608Metric, symbol Device:R_US
- C12: renamed from C35; footprint Capacitor_SMD:C_0402_1005Metric -> Capacitor_SMD:C_0603_1608Metric
- C13: renamed from C66; footprint Capacitor_SMD:C_0402_1005Metric -> Capacitor_SMD:C_0603_1608Metric
- C14: renamed from C67; footprint Capacitor_SMD:C_0402_1005Metric -> Capacitor_SMD:C_0603_1608Metric
- C15: renamed from C52; footprint Capacitor_SMD:C_0402_1005Metric -> Capacitor_SMD:C_0603_1608Metric
- C17: renamed from C83; footprint (none) -> Capacitor_SMD:C_0805_2012Metric
- C18: renamed from C82; footprint Capacitor_SMD:C_0603_1608Metric -> Capacitor_SMD:C_0805_2012Metric
- C19: renamed from C72; footprint Capacitor_SMD:C_0402_1005Metric -> Capacitor_SMD:C_0603_1608Metric
- C20: renamed from C73; footprint Capacitor_SMD:C_0402_1005Metric -> Capacitor_SMD:C_0603_1608Metric
- C22: renamed from C74; footprint Capacitor_SMD:C_0402_1005Metric -> Capacitor_SMD:C_0603_1608Metric
- C24: renamed from C75; footprint Capacitor_SMD:C_0402_1005Metric -> Capacitor_SMD:C_0603_1608Metric
- C27: renamed from C56; footprint Capacitor_SMD:C_0402_1005Metric -> Capacitor_SMD:C_0603_1608Metric
- C9: footprint (none) -> Capacitor_SMD:C_0805_2012Metric
- C9: footprint Capacitor_SMD:C_0402_1005Metric -> Capacitor_SMD:C_0603_1608Metric
- R14: renamed from R86; footprint Resistor_SMD:R_0402_1005Metric -> Resistor_SMD:R_0603_1608Metric
- R15: renamed from R42; footprint Resistor_SMD:R_0402_1005Metric -> Resistor_SMD:R_0603_1608Metric
- R17: renamed from R67; footprint Resistor_SMD:R_0402_1005Metric -> Resistor_SMD:R_0603_1608Metric
- R20: renamed from R45; footprint Resistor_SMD:R_0402_1005Metric -> Resistor_SMD:R_0603_1608Metric
- R21: renamed from R69; footprint Resistor_SMD:R_0402_1005Metric -> Resistor_SMD:R_0603_1608Metric
- R24: renamed from R77; footprint (none) -> Resistor_SMD:R_0603_1608Metric
- R25: renamed from R46; footprint (none) -> Resistor_SMD:R_0603_1608Metric
- R29: renamed from R87; footprint (none) -> Resistor_SMD:R_0603_1608Metric
- gave numbers to parts that had none: 2
- renumbered C80 to C25, C81 to C26, JP2 to JP1, L2 to L1, R72 to R16, SW2 to SW1, U14 to U6, U17 to U7, U15 to U8, Y2 to Y1
Connections:
- net +3V3: no longer U8.4 (PA03)
- net GND: now also C16.2, LED4.1 (K), Q6.4 (E1), R19.2, R22.2, R23.2, R30.1
- net TX: no longer U8.37 (PA18)
- net WDT_WDI: now also R26.2
- net MOSI: now reaches U8.38 (PA19)
- net PB07: now reaches U8.10 (PB07)
- net AIN3: now reaches U8.12 (PB09)
- net PB12: now reaches U8.25 (PB12)
- net PB13: now reaches U8.26 (PB13)
- net PB14: now reaches U8.27 (PB14)
- net PB15: now reaches U8.28 (PB15)
- net PA12: now reaches U8.29 (PA12)
- net PA13: now reaches U8.30 (PA13)
- net PA14: now reaches U8.31 (PA14)
- net PA15: now reaches U8.32 (PA15)
- net PA16: now reaches U8.35 (PA16)
- net SCK: now reaches U8.36 (PA17)
- net PA20: now reaches U8.41 (PA20)
- net HARD_RST: now reaches U8.43 (PA22)
- net PB04: now reaches U8.5 (PB04)
- net ~{FAULT}: now reaches U8.51 (PA27)
- net ~{FAULT}: now also R22.1, R31.2
- net PB30: now reaches U8.59 (PB30)
- net PB05: now reaches U8.6 (PB05)
- net PB31: now reaches U8.60 (PB31)
- net PB00: now reaches U8.61 (PB00)
- net PB01: now reaches U8.62 (PB01)
- net PB02: now reaches U8.63 (PB02)
- net PB06: now reaches U8.9 (PB06)
- net at D3.1 (DOUT): now also R30.2
- net AIN15 renamed PB03
- net AIN7 renamed VAA_ADC
- net VAA_ADC: now also C16.1, R18.2, R19.1
- new net: Q2.2 (B), R31.1
- new net: LED4.2 (A), R104.1
- new net: Q2.1 (C), R104.2
- new net: Q6.5 (B1), R27.1
- new net: Q6.2 (B2), R26.1
- new net: LED1.1 (K), Q6.6 (C2)
- new net: LED1.2 (A), R28.2
- new net: Q6.1 (E2), Q6.3 (C1)
- new net AIN1: U8.4 (PA03)
- new net LED_PWR: Q2.3 (E), R27.2, R28.1
- new net MISO: R23.1, U8.37 (PA18)
- new net VAA: R18.1
Other:
- note added: "ATSAMD51 MCU"
- note added: "SERCOM1 IOSET3"
- note added: "SERCOM3 IOSET3"
- note added: "SERCOM5 IOSET1"
- note added: "STATUS LEDs"
- note removed: "SERCOM1/IOSET3"
- note removed: "SERCOM5/IOSET1"
- note removed: "STATUS LED"
- moved on the sheet: C17, C18, C19, C20, C22, C24, C25, C26, C27, C9, D3, L1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

Commit message: working
Parts:
- removed Q2: PNP, symbol Simulation_SPICE:PNP
- added Q2: MMBT3906T, Package_TO_SOT_SMD:SOT-523, symbol Device:Q_PNP_BEC
Connections:
- net LED_PWR: now also Q2.2 (E)
- net at R31.1: now also Q2.1 (B)
- net at R104.2: now also Q2.3 (C)
Changed lines of the file:
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@@
-    )
-  )
-  (symbol (lib_id "Simulation_SPICE:PNP") (at 388.62 143.51 0) (mirror x) (unit 1)
-    (in_bom yes) (on_board yes) (dnp no) (fields_autoplaced)
-    (property "Reference" "Q2" (at 393.7 142.875 0)
-      (effects (font (size 1.27 1.27)) (justify left))
-    )
-    (property "Value" "PNP" (at 393.7 145.415 0)
-      (effects (font (size 1.27 1.27)) (justify left))
-    )
-    (property "Footprint" "" (at 424.18 143.51 0)
-      (effects (font (size 1.27 1.27)) hide)
-    )
-    (property "Datasheet" "~" (at 424.18 143.51 0)
-      (effects (font (size 1.27 1.27)) hide)
-    )
-    (property "Sim.Device" "PNP" (at 388.62 143.51 0)
-      (effects (font (size 1.27 1.27)) hide)
-    )
-    (property "Sim.Type" "GUMMELPOON" (at 388.62 143.51 0)
-      (effects (font (size 1.27 1.27)) hide)
-    )
-    (property "Sim.Pins" "1=C 2=B 3=E" (at 388.62 143.51 0)
-      (effects (font (size 1.27 1.27)) hide)
-    )
-    (pin "1")
-    (pin "2")
-    (pin "3")
-    (instances
-      (project "magnetotorqer-drive-board"
-        (path "/612afcad-8da9-4dff-bf3c-8828929809ff/0b2ade16-2e66-40b3-a5ca-aae3c5ec3394"
-          (reference "Q2") (unit 1)
-        )
-      )
     )
   )
@@
         )
       )
+    )
+  )
+  (symbol (lib_id "Device:Q_PNP_BEC") (at 388.62 143.51 0) (mirror x) (unit 1)
+    (in_bom yes) (on_board yes) (dnp no) (fields_autoplaced)
+    (property "Reference" "Q2" (at 393.7 142.875 0)
+      (effects (font (size 1.27 1.27)) (justify left))
+    )
+    (property "Value" "MMBT3906T" (at 393.7 145.415 0)
+      (effects (font (size 1.27 1.27)) (justify left))
+    )
+    (property "Footprint" "Package_TO_SOT_SMD:SOT-523" (at 393.7 146.05 0)
+      (effects (font (size 1.27 1.27)) hide)
+    )
+    (property "Datasheet" "https://www.diodes.com/assets/Datasheets/ds30271.pdf" (at 388.62 143.51 0)
+      (effects (font (size 1.27 1.27)) hide)
+    )
+    (property "Mfr. Part No" "MMBT3906T-7-F" (at 388.62 143.51 0)
+      (effects (font (size 1.27 1.27)) hide)
+    )
+    (property "Manufacturer" "Diodes Incorporated" (at 388.62 143.51 0)
+      (effects (font (size 1.27 1.27)) hide)
+    )
+    (property "Description" "TRANS PNP 40V 0.2A SOT523" (at 388.62 143.51 0)
+      (effects (font (size 1.27 1.27)) hide)
+    )
+    (pin "1")
+    (pin "2")
+    (pin "3")
+    (instances
+      (project "magnetotorqer-drive-board"
+        (path "/612afcad-8da9-4dff-bf3c-8828929809ff/0b2ade16-2e66-40b3-a5ca-aae3c5ec3394"
+          (reference "Q2") (unit 1)
+        )
+      )
+      (project "mainboard"
+        (path "/d1441985-7b63-4bf8-a06d-c70da2e3b78b/94774350-68be-4131-9d22-bdea2eae3261"
+          (reference "Q76") (unit 1)
+        )
+        (path "/d1441985-7b63-4bf8-a06d-c70da2e3b78b/00000000-0000-0000-0000-00005ede7915/16f74d99-fb34-4942-94f7-264307a230d0"
+          (reference "Q53") (unit 1)
+        )
+        (path "/d1441985-7b63-4bf8-a06d-c70da2e3b78b/00000000-0000-0000-0000-00005ede7915/8f80f71d-2dab-4aed-a364-86eb17282b90"
+          (reference "Q54") (unit 1)
+        )
+        (path "/d1441985-7b63-4bf8-a06d-c70da2e3b78b/00000000-0000-0000-0000-00005ede7915/f59d3a27-35da-42dd-8f28-13490a6a67ab"
+          (reference "Q55") (unit 1)
+        )
+        (path "/d1441985-7b63-4bf8-a06d-c70da2e3b78b/00000000-0000-0000-0000-00005ede7915/0be551f5-4cd0-4099-afa0-41f5d887dd91"
+          (reference "Q52") (unit 1)
+        )
+      )

Commit message: placement
Connections:
- net +3V3 renamed +3V3D
- net +3V3D: no longer C9.1, C9.1, U8.8 (VDDANA)
- new net +3V3A: C9.1, C9.1, U8.8 (VDDANA)
Changed lines of the file:
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@@
+      (effects (font (size 1.27 1.27)) hide)
+    )
+    (property "Manufacturer" "" (at 289.56 76.2 0)
+      (effects (font (size 1.27 1.27)) hide)
+    )
+    (property "Mfr. Part No" "" (at 289.56 76.2 0)
+      (effects (font (size 1.27 1.27)) hide)
+    )
+    (property "Description" "" (at 289.56 76.2 0)
       (effects (font (size 1.27 1.27)) hide)
     )
@@
     )
     (property "Datasheet" "" (at 44.45 64.77 0)
+      (effects (font (size 1.27 1.27)) hide)
+    )
+    (property "Manufacturer" "" (at 44.45 64.77 0)
+      (effects (font (size 1.27 1.27)) hide)
+    )
+    (property "Mfr. Part No" "" (at 44.45 64.77 0)
+      (effects (font (size 1.27 1.27)) hide)
+    )
+    (property "Description" "" (at 44.45 64.77 0)
       (effects (font (size 1.27 1.27)) hide)
     )
@@
     )
     (property "Datasheet" "" (at 78.74 128.27 0)
+      (effects (font (size 1.27 1.27)) hide)
+    )
+    (property "Manufacturer" "" (at 78.74 128.27 0)
+      (effects (font (size 1.27 1.27)) hide)
+    )
+    (property "Mfr. Part No" "" (at 78.74 128.27 0)
+      (effects (font (size 1.27 1.27)) hide)
+    )
+    (property "Description" "" (at 78.74 128.27 0)
       (effects (font (size 1.27 1.27)) hide)
     )
@@
       (effects (font (size 1.27 1.27)) hide)
     )
+    (property "Manufacturer" "" (at 93.98 160.02 0)
+      (effects (font (size 1.27 1.27)) hide)
+    )
+    (property "Mfr. Part No" "" (at 93.98 160.02 0)
+      (effects (font (size 1.27 1.27)) hide)
+    )
+    (property "Description" "" (at 93.98 160.02 0)
+      (effects (font (size 1.27 1.27)) hide)
+    )
     (pin "1")
     (instances
@@
       (effects (font (size 1.27 1.27)) hide)
     )
+    (property "Manufacturer" "" (at 153.67 171.45 0)
+      (effects (font (size 1.27 1.27)) hide)
+    )
+    (property "Mfr. Part No" "" (at 153.67 171.45 0)
+      (effects (font (size 1.27 1.27)) hide)
+    )
+    (property "Description" "" (at 153.67 171.45 0)
+      (effects (font (size 1.27 1.27)) hide)
+    )
     (pin "1")
     (instances
@@
       (effects (font (size 1.27 1.27)) hide)
     )
+    (property "Manufacturer" "" (at 265.43 76.2 0)
+      (effects (font (size 1.27 1.27)) hide)
+    )
+    (property "Mfr. Part No" "" (at 265.43 76.2 0)
+      (effects (font (size 1.27 1.27)) hide)
+    )
+    (property "Description" "" (at 265.43 76.2 0)
+      (effects (font (size 1.27 1.27)) hide)
+    )
     (pin "1")
     (instances
@@
     )
     (property "Datasheet" "" (at 256.54 96.52 0)
+      (effects (font (size 1.27 1.27)) hide)
+    )
+    (property "Manufacturer" "" (at 256.54 96.52 0)
+      (effects (font (size 1.27 1.27)) hide)
+    )
+    (property "Mfr. Part No" "" (at 256.54 96.52 0)
+      (effects (font (size 1.27 1.27)) hide)
+    )
+    (property "Description" "" (at 256.54 96.52 0)
       (effects (font (size 1.27 1.27)) hide)
     )
@@
       (effects (font (size 1.27 1.27)) hide)
     )
+    (property "Manufacturer" "" (at 96.52 205.74 0)
+      (effects (font (size 1.27 1.27)) hide)
+    )
+    (property "Mfr. Part No" "" (at 96.52 205.74 0)
+      (effects (font (size 1.27 1.27)) hide)
+    )
+    (property "Description" "" (at 96.52 205.74 0)
+      (effects (font (size 1.27 1.27)) hide)
+    )
     (pin "1")
     (instances
@@
       (effects (font (size 1.27 1.27)) hide)
     )
+    (property "Manufacturer" "" (at 53.34 127 0)
+      (effects (font (size 1.27 1.27)) hide)
+    )
+    (property "Mfr. Part No" "" (at 53.34 127 0)
+      (effects (font (size 1.27 1.27)) hide)
+    )
+    (property "Description" "" (at 53.34 127 0)
+      (effects (font (size 1.27 1.27)) hide)
+    )

Commit message: routing mostly complete
Parts:
- R26, R27, R31: footprint Resistor_SMD:R_0603_1608Metric -> Resistor_SMD:R_0402_1005Metric
Connections:
- net LED_PWR is gone; now on net LED_VCC: Q2.2 (E), R27.2, R28.1
- net PB03 renamed AIN15
Changed lines of the file:
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@@
     (effects (font (size 1.27 1.27)) (justify right bottom))
   )
-  (global_label "LED_PWR" (shape input) (at 370.84 132.08 180) (fields_autoplaced)
-    (effects (font (size 1.016 1.016)) (justify right))
-    (property "Intersheetrefs" "${INTERSHEET_REFS}" (at 362.3138 132.08 0)
-      (effects (font (size 1.016 1.016)) (justify right) hide)
-    )
-  )
-  (global_label "LED_PWR" (shape input) (at 317.5 171.45 180) (fields_autoplaced)
-    (effects (font (size 1.016 1.016)) (justify right))
-    (property "Intersheetrefs" "${INTERSHEET_REFS}" (at 308.9738 171.45 0)
-      (effects (font (size 1.016 1.016)) (justify right) hide)
+  (global_label "LED_VCC" (shape input) (at 317.5 171.45 180) (fields_autoplaced)
+    (effects (font (size 1.27 1.27)) (justify right))
+    (property "Intersheetrefs" "${INTERSHEET_REFS}" (at 307.2051 171.45 0)
+      (effects (font (size 1.27 1.27)) (justify right) hide)
     )
   )
@@
     )
   )
-  (global_label "LED_PWR" (shape input) (at 335.28 132.08 180) (fields_autoplaced)
-    (effects (font (size 1.016 1.016)) (justify right))
-    (property "Intersheetrefs" "${INTERSHEET_REFS}" (at 326.7538 132.08 0)
-      (effects (font (size 1.016 1.016)) (justify right) hide)
+  (global_label "LED_VCC" (shape input) (at 370.84 132.08 180) (fields_autoplaced)
+    (effects (font (size 1.27 1.27)) (justify right))
+    (property "Intersheetrefs" "${INTERSHEET_REFS}" (at 360.5451 132.08 0)
+      (effects (font (size 1.27 1.27)) (justify right) hide)
+    )
+  )
+  (global_label "LED_VCC" (shape input) (at 335.28 132.08 180) (fields_autoplaced)
+    (effects (font (size 1.27 1.27)) (justify right))
+    (property "Intersheetrefs" "${INTERSHEET_REFS}" (at 324.9851 132.08 0)
+      (effects (font (size 1.27 1.27)) (justify right) hide)
     )
   )
@@
     (effects (font (size 1.27 1.27)) (justify right))
   )
-  (hierarchical_label "PB03" (shape bidirectional) (at 265.43 121.92 0) (fields_autoplaced)
+  (hierarchical_label "AIN15" (shape input) (at 265.43 121.92 0) (fields_autoplaced)
     (effects (font (size 1.27 1.27)) (justify left))
   )
@@
       (effects (font (size 1.27 1.27)))
     )
-    (property "Footprint" "Resistor_SMD:R_0603_1608Metric" (at 376.936 144.526 90)
+    (property "Footprint" "Resistor_SMD:R_0402_1005Metric" (at 376.936 144.526 90)
       (effects (font (size 1.27 1.27)) hide)
     )
@@
       (effects (font (size 1.27 1.27)))
     )
-    (property "Footprint" "Resistor_SMD:R_0603_1608Metric" (at 323.596 172.466 90)
+    (property "Footprint" "Resistor_SMD:R_0402_1005Metric" (at 323.596 172.466 90)
       (effects (font (size 1.27 1.27)) hide)
     )
@@
       (effects (font (size 1.27 1.27)))
     )
-    (property "Footprint" "Resistor_SMD:R_0603_1608Metric" (at 323.596 158.496 90)
-      (effects (font (size 1.27 1.27)) hide)
-    )
+    (property "Footprint" "Resistor_SMD:R_0402_1005Metric" (at 323.596 158.496 90)
+      (effects (font (size 1.27 1.27)) hide)
+    )
