File: revA/control.kicad_sch (KiCad schematic)
At the start: 49 parts, among them J8 Conn_01x06, P2 FTSH-105-01-F-DV-K-TR, Q2 MMBT3906T, Q6 MMDT2222A, SW1 KMR231NG LFS, U6 MR25H10MDF, U7 MAX708RESA-T, U8 ATSAMD51J20A-A, Y1 32.768kHz

Commit message: working
Parts:
- removed J8: Conn_01x06, Connector_PinHeader_2.54mm:PinHeader_1x06_P2.54mm_Vertical_SMD_Pin1Right, symbol Connector_Generic:Conn_01x06
- added R22, R25: 0, Resistor_SMD:R_0603_1608Metric, symbol Device:R_US
- C12: renamed from C13; Manufacturer TDK -> (none); Mfr. Part No CGA2B2NP01H080D050BA -> (none)
- C13: renamed from C14; Manufacturer TDK -> (none); Mfr. Part No CGA2B2NP01H080D050BA -> (none)
- C14: renamed from C12; Manufacturer TDK -> (none); Mfr. Part No CGA2B3X7R1H104K050BE -> (none)
- C15: renamed from C19; Manufacturer TDK -> (none); Mfr. Part No CGA2B3X7R1H104K050BE -> (none)
- C16: renamed from C20; Manufacturer TDK -> (none); Mfr. Part No CGA2B3X7R1H104K050BE -> (none)
- C17: renamed from C22; Manufacturer TDK -> (none); Mfr. Part No CGA2B3X7R1H104K050BE -> (none)
- C18: renamed from C24; Manufacturer TDK -> (none); Mfr. Part No CGA2B3X7R1H104K050BE -> (none)
- C19: renamed from C25; Manufacturer TDK -> (none); Mfr. Part No CGA4J1X7S1E106K125AE -> (none)
- C20: renamed from C26; Manufacturer TDK -> (none); Mfr. Part No CGA4J1X7S1E106K125AE -> (none)
- C21: renamed from C27; Manufacturer TDK -> (none); Mfr. Part No CGA2B3X7R1H104K050BE -> (none)
- C26: renamed from C16; Manufacturer TDK -> (none); Mfr. Part No CGA2B3X7R1H104K050BE -> (none)
- C27: renamed from C15; Manufacturer TDK -> (none); Mfr. Part No CGA2B3X7R1H104K050BE -> (none)
- C9: Manufacturer TDK -> (none); Mfr. Part No CGA2B3X7R1H104K050BE -> (none)
- renumbered C17 to C22, C18 to C23, P2 to P3, Q2 to Q1, R29 to R16, R30 to R17, R28 to R20, R31 to R21, R24 to R23, R25 to R26, R26 to R27, R17 to R28, R16 to R29, R20 to R30, R27 to R31, R21 to R32, R22 to R33, R23 to R34, R14 to R35, U8 to U7, U7 to U8
Connections:
- net TX: now also R22.2; no longer U7.39 (PB16)
- net TX_DEBUG: now also R25.2; no longer U7.49 (PB22)
- new net: R22.1, U7.39 (PB16)
- new net: R25.1, U7.49 (PB22)
Other:
- note added: "YELLOW = WDI (blinks for heartbeat) RED = FAULT"
- note removed: "Debug Serial Header"
- title: (none) -> SCHEMATIC, CUBESAT MAGNETORQER DRIVER
- moved on the sheet: C12, C13, C14, C27, JP1, LED1, LED4, P3, Q1, Q6A, Q6B, R104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

Commit message: worked review changes
Parts:
- C27: renamed from C14; Manufacturer (none) -> TDK Corporation; Mfr. Part No (none) -> CGA3E2X7R1H104K080AE; Value2 (none) -> 50V
- C28: renamed from C12; footprint Capacitor_SMD:C_0603_1608Metric -> Capacitor_SMD:C_0402_1005Metric; Manufacturer (none) -> TDK Corporation; Mfr. Part No (none) -> CGA2B2NP01H080D050BA; Value2 (none) -> 50V
- C29: renamed from C13; footprint Capacitor_SMD:C_0603_1608Metric -> Capacitor_SMD:C_0402_1005Metric; Manufacturer (none) -> TDK Corporation; Mfr. Part No (none) -> CGA2B2NP01H080D050BA; Value2 (none) -> 50V
- C30: renamed from C27; Manufacturer (none) -> TDK Corporation; Mfr. Part No (none) -> CGA3E2X7R1H104K080AE; Value2 (none) -> 50V
- C31: renamed from C26; Manufacturer (none) -> TDK Corporation; Mfr. Part No (none) -> CGA3E2X7R1H104K080AE; Value2 (none) -> 50V
- C32: renamed from C22; Manufacturer (none) -> TDK Corporation; Mfr. Part No (none) -> CGA4J1X7S1E106K125AE; Value2 (none) -> 25V
- C33: renamed from C23; Manufacturer (none) -> TDK Corporation; Mfr. Part No (none) -> CGA4J3X7R1H105K125AE; Value2 (none) -> 50V
- C34: renamed from C15; Manufacturer (none) -> TDK Corporation; Mfr. Part No (none) -> CGA3E2X7R1H104K080AE; Value2 (none) -> 50V
- C35: renamed from C16; Manufacturer (none) -> TDK Corporation; Mfr. Part No (none) -> CGA3E2X7R1H104K080AE; Value2 (none) -> 50V
- C37: renamed from C17; Manufacturer (none) -> TDK Corporation; Mfr. Part No (none) -> CGA3E2X7R1H104K080AE; Value2 (none) -> 50V
- C39: renamed from C18; Manufacturer (none) -> TDK Corporation; Mfr. Part No (none) -> CGA3E2X7R1H104K080AE; Value2 (none) -> 50V
- C40: renamed from C19; Manufacturer (none) -> TDK Corporation; Mfr. Part No (none) -> CGA4J1X7S1E106K125AE; Value2 (none) -> 25V
- C41: renamed from C20; Manufacturer (none) -> TDK Corporation; Mfr. Part No (none) -> CGA4J1X7S1E106K125AE; Value2 (none) -> 25V
- C42: renamed from C21; Manufacturer (none) -> TDK Corporation; Mfr. Part No (none) -> CGA3E2X7R1H104K080AE; Value2 (none) -> 50V
- C?: renamed from C9; Manufacturer (none) -> TDK Corporation; Mfr. Part No (none) -> CGA4J1X7S1E106K125AE; Value2 (none) -> 25V
- C?: renamed from C9; Manufacturer (none) -> TDK Corporation; Mfr. Part No (none) -> CGA3E2X7R1H104K080AE; Value2 (none) -> 50V
- D5: renamed from D3; Manufacturer (none) -> Adafruit Industries LLC; Mfr. Part No (none) -> 2659
- LED?: renamed from LED4; Mfr. Part No APA2107LSECK -> APA2107LSECK/J3-PRV
- Q? (x2): renamed from Q6; Manufacturer (none) -> Diodes Incorporated; Mfr. Part No (none) -> MMDT2222A-7-F
- R34: renamed from R35; Manufacturer (none) -> Stackpole Electronics Inc; Mfr. Part No (none) -> RMCF0603FT10K0; Value2 (none) -> 100mW
- R35: renamed from R29; Manufacturer (none) -> Stackpole Electronics Inc; Mfr. Part No (none) -> RMCF0603FT330R; Value2 (none) -> 100mW
- R36: renamed from R15; Manufacturer (none) -> Stackpole Electronics Inc; Mfr. Part No (none) -> RMCF0603FT10K0; Value2 (none) -> 100mW
- R37: renamed from R28; Manufacturer (none) -> Stackpole Electronics Inc; Mfr. Part No (none) -> RMCF0603FT10K0; Value2 (none) -> 100mW
- R38: renamed from R18; Manufacturer (none) -> Stackpole Electronics Inc; Mfr. Part No (none) -> RMCF0603FT330K; Value2 (none) -> 100mW
- R39: renamed from R19; Manufacturer (none) -> Stackpole Electronics Inc; Mfr. Part No (none) -> RMCF0603FT110K; Value2 (none) -> 100mW
- R40: renamed from R30; Manufacturer (none) -> Stackpole Electronics Inc; Mfr. Part No (none) -> RMCF0603FT10K0; Value2 (none) -> 100mW
- R41: renamed from R32; Manufacturer (none) -> Stackpole Electronics Inc; Mfr. Part No (none) -> RMCF0603FT10K0; Value2 (none) -> 100mW
- R42: renamed from R33; Manufacturer (none) -> Stackpole Electronics Inc; Mfr. Part No (none) -> RMCF0603FT10K0; Value2 (none) -> 100mW
- R43: renamed from R34; Manufacturer (none) -> Stackpole Electronics Inc; Mfr. Part No (none) -> RMCF0603FT100K; Value2 (none) -> 100mW
- R44: renamed from R22; Manufacturer (none) -> Stackpole Electronics Inc; Mfr. Part No (none) -> RMCF0603ZT0R00; Value2 (none) -> 100mW
- R45: renamed from R23; Manufacturer (none) -> Stackpole Electronics Inc; Mfr. Part No (none) -> RMCF0603FG1K00; Value2 (none) -> 100mW
- R46: renamed from R25; Manufacturer (none) -> Stackpole Electronics Inc; Mfr. Part No (none) -> RMCF0603ZT0R00; Value2 (none) -> 100mW
- R47: renamed from R26; Manufacturer (none) -> Stackpole Electronics Inc; Mfr. Part No (none) -> RMCF0603FG1K00; Value2 (none) -> 100mW
- R48: renamed from R27; Manufacturer (none) -> Stackpole Electronics Inc; Mfr. Part No (none) -> RMCF0402FT10K0; Value2 (none) -> 62.5mW
- R49: renamed from R31; Manufacturer (none) -> Stackpole Electronics Inc; Mfr. Part No (none) -> RMCF0402FT10K0; Value2 (none) -> 62.5mW
- R50: renamed from R20; Manufacturer Stackpole Electronics -> Stackpole Electronics Inc; Value2 (none) -> 62.5mW
- R51: renamed from R16; value 499 -> 1k; Manufacturer (none) -> Stackpole Electronics Inc; Mfr. Part No (none) -> RMCF0603FG1K00; Value2 (none) -> 100mW
- R52: renamed from R21; Manufacturer (none) -> Stackpole Electronics Inc; Mfr. Part No (none) -> RMCF0402FT10K0; Value2 (none) -> 62.5mW
- R53: renamed from R17; Manufacturer (none) -> Stackpole Electronics Inc; Mfr. Part No (none) -> RMCF0603FT10K0; Value2 (none) -> 100mW
- R?: renamed from R104; Manufacturer (none) -> Stackpole Electronics Inc; Mfr. Part No (none) -> RMCF0402FT1K50; Value2 (none) -> 62.5mW
- SW1: Value2 (none) -> 50mA
- U10: renamed from U8; value MAX708RESA-T -> MAX708RESA+T; symbol SierraLobo:MAX708RESA-T -> SierraLobo:MAX708RESA; Mfr. Part No MAX708RESA-T -> MAX708RESA+T
- U12: renamed from U7; value ATSAMD51J20A-A -> ATSAMD51J20A-AU; symbol MCU_Microchip_SAMD:ATSAMD51J20A-A -> SierraLobo:ATSAMD51J20A-AU; Manufacturer (none) -> Microchip Technology; Mfr. Part No. (none) -> ATSAMD51J20A-AU
- renumbered LED1 to LED3, P3 to P4, Q1 to Q9, U6 to U11
