File: revA/driver.kicad_sch (KiCad schematic)
At the start: 17 parts, among them U5 TLV4110xDGN, U6 DRV8838DSGT, U7 INA199A2xDCK

Commit message: working
Parts:
- removed C20: 10uF, Capacitor_SMD:C_0805_2012Metric, symbol Device:C
- removed C21, C22, C24: 0.1uF, Capacitor_SMD:C_0402_1005Metric, symbol Device:C
- removed C23: 0.01uF, Capacitor_SMD:C_0402_1005Metric, symbol Device:C
- removed D2: SP1326-01LTG, Diode_SMD:D_SOD-523, symbol Device:D_TVS
- removed R15, R18: 110k, Resistor_SMD:R_0603_1608Metric, symbol Device:R_US
- removed R16, R20, R22: 1k, Resistor_SMD:R_0402_1005Metric, symbol Device:R_US
- removed R17, R21: 100k, Resistor_SMD:R_0402_1005Metric, symbol Device:R_US
- removed U5: TLV4110xDGN, Package_SO:MSOP-8-1EP_3x3mm_P0.65mm_EP1.68x1.88mm, symbol SierraLobo:TLV4110xDGN
- removed U6: DRV8838DSGT, Package_SON:WSON-8-1EP_2x2mm_P0.5mm_EP0.9x1.6mm, symbol magnetotorquer-test-board:DRV8838DSGT
- removed U7: INA199A2xDCK, Package_TO_SOT_SMD:SOT-363_SC-70-6, symbol Amplifier_Current:INA199xxDCK
- R19: value 1k -> ${R_sense}; footprint Resistor_SMD:R_0402_1005Metric -> (none); Manufacturer (none) -> ${R_Sense Mfr}; Mfr. Part No (none) -> ${R_Sense Part No}
Connections:
- net OUT2: now also R19.2
- net ~{HB_SLEEP}: no longer R19.1
- new net OUT2_SEN: R19.1
Other:
- added sheet Adjustable Buck Regulator 1 (adj_buck.kicad_sch)
- added sheet Current Feedback 1 (i_fb.kicad_sch)
- added sheet H-Bridge 1 (h_bridge.kicad_sch)
- note added: "MTQ DRIVER"
- note added: "X/Y MTQ 80-145R, 0.2W 50mA MAX Z MTQ 30-55R, 0.57W 137mA MAX Control of VDRV is 0-5V so control can exceed max power of MTQs."
- note removed: "100v/v gain"
- note removed: "Amplify DAC power output"
- note removed: "CURRENT SENSE AMP"
- note removed: "DAC_IN = 0-5V X/Y MTQ resistance = 80-145R, 0.2W rated Z MTQ resistance = 30-55R, 0.57W Maximum output current control should be limited by MTQ power (0.2W) -> Ioutmax(X,Y) = 50mA (80R, 0.2W) -> Ioutmax(Z) = 137mA (30R, 0.57W)"
- note removed: "FET Back diodes in full bridge should clamp drive voltage"
- note removed: "HALF BRIDGE DRIVER"
- note removed: "POWER AMP"
- note removed: "Select Rsense to give 1.5V deflection at Imax"
- note removed: "Sense resistor at higher level sheet"
- note removed: "VMID is mid-supply of VADC (1.65V)"
- note removed: "current sense amplifier"
- note removed: "for bi-directional control"
- note removed: "read current output"

Commit message: working
Parts:
- added TP3 (x3), TP4: ${NET_NAME(1)}, TestPoint:TestPoint_Keystone_5000-5004_Miniature, symbol Connector:TestPoint
- R8: renamed from R19; footprint (none) -> Resistor_SMD:R_0603_1608Metric
Connections:
- net OUT1: now also TP3.1
- net OUT2: now also TP3.1
- net V_RSEN: now also TP3.1
- new net GND: TP4.1
Other:
- note added: "TEST POINTS"

Commit message: placement
Parts:
- removed TP4: ${NET_NAME(1)}, TestPoint:TestPoint_Keystone_5000-5004_Miniature, symbol Connector:TestPoint
- R8: footprint Resistor_SMD:R_0603_1608Metric -> Resistor_SMD:R_0805_2012Metric
Connections:
- net OUT1: now also R8.2
- net OUT2: no longer R8.2
- net OUT2_SEN renamed OUT1_SEN
Other:
- moved on the sheet: R8
Changed lines of the file:
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@@
 (kicad_sch (version 20230121) (generator eeschema)
   (paper "B")
-  (junction (at 262.89 119.38) (diameter 0) (color 0 0 0 0)
-  )
-  (junction (at 273.05 119.38) (diameter 0) (color 0 0 0 0)
+  (junction (at 262.89 115.57) (diameter 0) (color 0 0 0 0)
+  )
+  (junction (at 273.05 115.57) (diameter 0) (color 0 0 0 0)
   )
   (wire (pts (xy 162.56 115.57) (xy 203.2 115.57))
@@
     (stroke (width 0) (type default))
   )
+  (wire (pts (xy 220.98 119.38) (xy 294.64 119.38))
+    (stroke (width 0) (type default))
+  )
   (wire (pts (xy 203.2 128.27) (xy 185.42 128.27))
     (stroke (width 0) (type default))
@@
     (stroke (width 0) (type default))
   )
-  (wire (pts (xy 220.98 115.57) (xy 294.64 115.57))
+  (wire (pts (xy 271.78 115.57) (xy 273.05 115.57))
+    (stroke (width 0) (type default))
+  )
+  (wire (pts (xy 220.98 115.57) (xy 262.89 115.57))
     (stroke (width 0) (type default))
   )
@@
     (stroke (width 0) (type default))
   )
-  (wire (pts (xy 273.05 119.38) (xy 294.64 119.38))
-    (stroke (width 0) (type default))
-  )
   (wire (pts (xy 124.46 123.19) (xy 137.16 123.19))
     (stroke (width 0) (type default))
   )
-  (wire (pts (xy 262.89 119.38) (xy 262.89 130.81))
-    (stroke (width 0) (type default))
-  )
-  (wire (pts (xy 273.05 119.38) (xy 271.78 119.38))
-    (stroke (width 0) (type default))
-  )
-  (wire (pts (xy 332.74 142.24) (xy 345.44 142.24))
+  (wire (pts (xy 262.89 115.57) (xy 262.89 130.81))
     (stroke (width 0) (type default))
   )
@@
     (stroke (width 0) (type default))
   )
-  (wire (pts (xy 273.05 130.81) (xy 273.05 119.38))
-    (stroke (width 0) (type default))
-  )
-  (wire (pts (xy 264.16 119.38) (xy 262.89 119.38))
-    (stroke (width 0) (type default))
-  )
-  (wire (pts (xy 220.98 119.38) (xy 262.89 119.38))
+  (wire (pts (xy 262.89 115.57) (xy 264.16 115.57))
+    (stroke (width 0) (type default))
+  )
+  (wire (pts (xy 273.05 115.57) (xy 273.05 130.81))
+    (stroke (width 0) (type default))
+  )
+  (wire (pts (xy 273.05 115.57) (xy 294.64 115.57))
     (stroke (width 0) (type default))
   )
@@
     (effects (font (size 1.27 1.27)) (justify left bottom))
   )
-  (label "OUT2_SEN" (at 234.95 119.38 0) (fields_autoplaced)
+  (label "OUT1_SEN" (at 236.22 115.57 0) (fields_autoplaced)
     (effects (font (size 1.27 1.27)) (justify left bottom))
   )
@@
     )
   )
-  (symbol (lib_id "Device:R_US") (at 267.97 119.38 90) (unit 1)
+  (symbol (lib_id "Device:R_US") (at 267.97 115.57 90) (unit 1)
     (in_bom yes) (on_board yes) (dnp no) (fields_autoplaced)
-    (property "Reference" "R8" (at 267.97 123.19 90)
-      (effects (font (size 1.27 1.27)))
-    )
-    (property "Value" "${R_sense}" (at 267.97 125.73 90)
-      (effects (font (size 1.27 1.27)))
-    )
-    (property "Footprint" "Resistor_SMD:R_0603_1608Metric" (at 268.224 118.364 90)
-      (effects (font (size 1.27 1.27)) hide)
-    )
-    (property "Datasheet" "~" (at 267.97 119.38 0)
-      (effects (font (size 1.27 1.27)) hide)
-    )
-    (property "Manufacturer" "${R_Sense Mfr}" (at 267.97 119.38 0)
-      (effects (font (size 1.27 1.27)) hide)
-    )
-    (property "Mfr. Part No" "${R_Sense Part No}" (at 267.97 119.38 0)
-      (effects (font (size 1.27 1.27)) hide)
-    )
-    (property "Description" "" (at 267.97 119.38 0)
+    (property "Reference" "R8" (at 267.97 110.49 90)
+      (effects (font (size 1.27 1.27)))
+    )
+    (property "Value" "${R_sense}" (at 267.97 113.03 90)
+      (effects (font (size 1.27 1.27)))
+    )
+    (property "Footprint" "Resistor_SMD:R_0805_2012Metric" (at 268.224 114.554 90)
+      (effects (font (size 1.27 1.27)) hide)
+    )
+    (property "Datasheet" "~" (at 267.97 115.57 0)
+      (effects (font (size 1.27 1.27)) hide)
+    )
+    (property "Manufacturer" "${R_Sense Mfr}" (at 267.97 115.57 0)
+      (effects (font (size 1.27 1.27)) hide)
+    )
+    (property "Mfr. Part No" "${R_Sense Part No}" (at 267.97 115.57 0)
+      (effects (font (size 1.27 1.27)) hide)
+    )
+    (property "Description" "" (at 267.97 115.57 0)
       (effects (font (size 1.27 1.27)) hide)
     )
@@
     )
   )
-  (symbol (lib_id "Connector:TestPoint") (at 345.44 142.24 0) (unit 1)
-    (in_bom yes) (on_board yes) (dnp no)
-    (property "Reference" "TP4" (at 347.98 138.303 0)
-      (effects (font (size 1.27 1.27)) (justify left))
-    )
-    (property "Value" "${NET_NAME(1)}" (at 347.98 140.843 0)
-      (effects (font (size 1.27 1.27)) (justify left) hide)
-    )
-    (property "Footprint" "TestPoint:TestPoint_Keystone_5000-5004_Miniature" (at 350.52 142.24 0)
-      (effects (font (size 1.27 1.27)) hide)
-    )
-    (property "Datasheet" "https://www.keyelco.com/userAssets/file/M65p56.pdf" (at 350.52 142.24 0)
-      (effects (font (size 1.27 1.27)) hide)
-    )
-    (property "Manufacturer" "Keystone" (at 345.44 142.24 0)
-      (effects (font (size 1.27 1.27)) hide)
-    )
-    (property "Mfr. Part No" "5001" (at 350.52 140.97 0)
-      (effects (font (size 1.27 1.27)))
-    )
-    (property "Description" "PC TEST POINT MINIATURE BLACK" (at 345.44 142.24 0)
-      (effects (font (size 1.27 1.27)) hide)
-    )
-    (pin "1")
-    (instances
-      (project "magnetotorqer-drive-board"
-        (path "/612afcad-8da9-4dff-bf3c-8828929809ff/8ccdbec3-7661-4a0b-9858-5169c364aebb/765443f8-c18e-4cd2-97d5-a5c0f8a3785d"
-          (reference "TP4") (unit 1)
-        )
-        (path "/612afcad-8da9-4dff-bf3c-8828929809ff/8ccdbec3-7661-4a0b-9858-5169c364aebb/5c5f6184-6b4f-4d2f-a4ab-4cc197c5e0c0"
-          (reference "TP18") (unit 1)
-        )
-        (path "/612afcad-8da9-4dff-bf3c-8828929809ff/0c4bd054-86d6-4fc6-b8bd-5dc40d9d4357/5c5f6184-6b4f-4d2f-a4ab-4cc197c5e0c0"
-          (reference "TP13") (unit 1)
-        )
-        (path "/612afcad-8da9-4dff-bf3c-8828929809ff/853a01c4-0f0d-42ee-a9e8-050403071668/5c5f6184-6b4f-4d2f-a4ab-4cc197c5e0c0"
-          (reference "TP27") (unit 1)
-        )
-        (path "/612afcad-8da9-4dff-bf3c-8828929809ff/8ccdbec3-7661-4a0b-9858-5169c364aebb"
-          (reference "TP4") (unit 1)
-        )
-        (path "/612afcad-8da9-4dff-bf3c-8828929809ff/0c4bd054-86d6-4fc6-b8bd-5dc40d9d4357"
-          (reference "TP8") (unit 1)
-        )
-        (path "/612afcad-8da9-4dff-bf3c-8828929809ff/853a01c4-0f0d-42ee-a9e8-050403071668"
-          (reference "TP17") (unit 1)
-        )
-      )
-    )
-  )
   (symbol (lib_id "Connector:TestPoint") (at 345.44 135.89 0) (unit 1)
     (in_bom yes) (on_board yes) (dnp no)
@@
         )
       )
-    )
-  )
-  (symbol (lib_id "power:GND") (at 332.74 142.24 0) (unit 1)
-    (in_bom yes) (on_board yes) (dnp no) (fields_autoplaced)
-    (property "Reference" "#PWR037" (at 332.74 148.59 0)
-      (effects (font (size 1.27 1.27)) hide)
-    )
-    (property "Value" "GND" (at 332.74 146.8025 0)
-      (effects (font (size 1.27 1.27)))
-    )
-    (property "Footprint" "" (at 332.74 142.24 0)
-      (effects (font (size 1.27 1.27)) hide)
-    )
-    (property "Datasheet" "" (at 332.74 142.24 0)
-      (effects (font (size 1.27 1.27)) hide)
-    )
-    (pin "1")
-    (instances
-      (project "magnetotorqer-drive-board"
-        (path "/612afcad-8da9-4dff-bf3c-8828929809ff/8ccdbec3-7661-4a0b-9858-5169c364aebb"
-          (reference "#PWR037") (unit 1)
-        )
-        (path "/612afcad-8da9-4dff-bf3c-8828929809ff/8ccdbec3-7661-4a0b-9858-5169c364aebb/765443f8-c18e-4cd2-97d5-a5c0f8a3785d"
-          (reference "#PWR0104") (unit 1)
-        )
-        (path "/612afcad-8da9-4dff-bf3c-8828929809ff/8ccdbec3-7661-4a0b-9858-5169c364aebb/5c5f6184-6b4f-4d2f-a4ab-4cc197c5e0c0"
-          (reference "#PWR0117") (unit 1)
-        )
-        (path "/612afcad-8da9-4dff-bf3c-8828929809ff/0c4bd054-86d6-4fc6-b8bd-5dc40d9d4357/5c5f6184-6b4f-4d2f-a4ab-4cc197c5e0c0"
-          (reference "#PWR099") (unit 1)
-        )
-        (path "/612afcad-8da9-4dff-bf3c-8828929809ff/853a01c4-0f0d-42ee-a9e8-050403071668/5c5f6184-6b4f-4d2f-a4ab-4cc197c5e0c0"
-          (reference "#PWR0148") (unit 1)
-        )
-        (path "/612afcad-8da9-4dff-bf3c-8828929809ff/0c4bd054-86d6-4fc6-b8bd-5dc40d9d4357"
-          (reference "#PWR038") (unit 1)
-        )
-        (path "/612afcad-8da9-4dff-bf3c-8828929809ff/853a01c4-0f0d-42ee-a9e8-050403071668"
-          (reference "#PWR0103") (unit 1)
-        )
-      )
-      (project "payload-interface-board"
-        (path "/dc2801a1-d539-4721-b31f-fe196b9f13df/24d21d3f-37df-43db-a302-5a6c43abae48/9a405ebb-5c40-4de0-9346-a2ae3aaabc82"
-          (reference "#PWR053") (unit 1)
-        )
-        (path "/dc2801a1-d539-4721-b31f-fe196b9f13df/24d21d3f-37df-43db-a302-5a6c43abae48/146b684a-f73b-4eb1-adfe-30f1964810bc"
-          (reference "#PWR071") (unit 1)
-        )
-        (path "/dc2801a1-d539-4721-b31f-fe196b9f13df/24d21d3f-37df-43db-a302-5a6c43abae48/d37b3655-4247-47b6-9578-a41f570787b9"
-          (reference "#PWR063") (unit 1)
-        )
-      )

Commit message: routing mostly complete
Parts:
- TP3: footprint TestPoint:TestPoint_Keystone_5000-5004_Miniature -> SierraLobo:TestPoint_Keystone_5000-5004_Miniature
Changed lines of the file:
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@@
       (effects (font (size 1.27 1.27)) (justify left) hide)
     )
-    (property "Footprint" "TestPoint:TestPoint_Keystone_5000-5004_Miniature" (at 350.52 128.27 0)
+    (property "Footprint" "SierraLobo:TestPoint_Keystone_5000-5004_Miniature" (at 350.52 128.27 0)
       (effects (font (size 1.27 1.27)) hide)
     )
@@
       (effects (font (size 1.27 1.27)) (justify left) hide)
     )
-    (property "Footprint" "TestPoint:TestPoint_Keystone_5000-5004_Miniature" (at 350.52 120.65 0)
+    (property "Footprint" "SierraLobo:TestPoint_Keystone_5000-5004_Miniature" (at 350.52 120.65 0)
       (effects (font (size 1.27 1.27)) hide)
     )
@@
       (effects (font (size 1.27 1.27)) (justify left) hide)
     )
-    (property "Footprint" "TestPoint:TestPoint_Keystone_5000-5004_Miniature" (at 350.52 135.89 0)
+    (property "Footprint" "SierraLobo:TestPoint_Keystone_5000-5004_Miniature" (at 350.52 135.89 0)
       (effects (font (size 1.27 1.27)) hide)
     )

Commit message: working
Parts:
- R9: renamed from R8; value ${R_sense} -> ${R_Sense}
- TP3: Mfr. Part No 5119 -> 5002
Other:
- title: (none) -> SCHEMATIC, CUBESAT MAGNETORQER DRIVER
Changed lines of the file:
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@@
 (kicad_sch (version 20230121) (generator eeschema)
   (paper "B")
+  (title_block
+    (title "SCHEMATIC, CUBESAT MAGNETORQER DRIVER")
+    (date "2023-06-28")
+    (rev "A")
+    (comment 1 "CH")
+    (comment 2 "CH")
+    (comment 3 "RD21-6005")
+  )
   (junction (at 262.89 115.57) (diameter 0) (color 0 0 0 0)
   )
@@
       (effects (font (size 1.27 1.27)) hide)
     )
-    (property "Mfr. Part No" "5119" (at 350.52 127 0)
+    (property "Mfr. Part No" "5002" (at 350.52 127 0)
       (effects (font (size 1.27 1.27)))
     )
-    (property "Description" "PC TEST POINT MINIATURE PURPLE" (at 345.44 128.27 0)
+    (property "Description" "PC TEST POINT MINIATURE WHITE" (at 345.44 128.27 0)
       (effects (font (size 1.27 1.27)) hide)
     )
@@
         )
         (path "/612afcad-8da9-4dff-bf3c-8828929809ff/8ccdbec3-7661-4a0b-9858-5169c364aebb"
-          (reference "TP2") (unit 1)
+          (reference "TP10") (unit 1)
         )
         (path "/612afcad-8da9-4dff-bf3c-8828929809ff/0c4bd054-86d6-4fc6-b8bd-5dc40d9d4357"
-          (reference "TP6") (unit 1)
+          (reference "TP13") (unit 1)
         )
         (path "/612afcad-8da9-4dff-bf3c-8828929809ff/853a01c4-0f0d-42ee-a9e8-050403071668"
-          (reference "TP15") (unit 1)
+          (reference "TP21") (unit 1)
         )
       )
@@
       (effects (font (size 1.27 1.27)) hide)
     )
-    (property "Mfr. Part No" "5119" (at 350.52 119.38 0)
+    (property "Mfr. Part No" "5002" (at 350.52 119.38 0)
       (effects (font (size 1.27 1.27)))
     )
-    (property "Description" "PC TEST POINT MINIATURE PURPLE" (at 345.44 120.65 0)
+    (property "Description" "PC TEST POINT MINIATURE WHITE" (at 345.44 120.65 0)
       (effects (font (size 1.27 1.27)) hide)
     )
@@
         )
         (path "/612afcad-8da9-4dff-bf3c-8828929809ff/8ccdbec3-7661-4a0b-9858-5169c364aebb"
-          (reference "TP1") (unit 1)
+          (reference "TP9") (unit 1)
         )
         (path "/612afcad-8da9-4dff-bf3c-8828929809ff/0c4bd054-86d6-4fc6-b8bd-5dc40d9d4357"
-          (reference "TP5") (unit 1)
+          (reference "TP12") (unit 1)
         )
         (path "/612afcad-8da9-4dff-bf3c-8828929809ff/853a01c4-0f0d-42ee-a9e8-050403071668"
-          (reference "TP14") (unit 1)
+          (reference "TP20") (unit 1)
         )
       )
@@
   (symbol (lib_id "Device:R_US") (at 267.97 115.57 90) (unit 1)
     (in_bom yes) (on_board yes) (dnp no) (fields_autoplaced)
-    (property "Reference" "R8" (at 267.97 110.49 90)
+    (property "Reference" "R9" (at 267.97 110.49 90)
       (effects (font (size 1.27 1.27)))
     )
-    (property "Value" "${R_sense}" (at 267.97 113.03 90)
+    (property "Value" "${R_Sense}" (at 267.97 113.03 90)
       (effects (font (size 1.27 1.27)))
     )
@@
       (project "magnetotorqer-drive-board"
         (path "/612afcad-8da9-4dff-bf3c-8828929809ff/8ccdbec3-7661-4a0b-9858-5169c364aebb"
-          (reference "R8") (unit 1)
+          (reference "R9") (unit 1)
         )
         (path "/612afcad-8da9-4dff-bf3c-8828929809ff/0c4bd054-86d6-4fc6-b8bd-5dc40d9d4357"
-          (reference "R9") (unit 1)
+          (reference "R10") (unit 1)
         )
         (path "/612afcad-8da9-4dff-bf3c-8828929809ff/853a01c4-0f0d-42ee-a9e8-050403071668"
-          (reference "R46") (unit 1)
+          (reference "R50") (unit 1)
         )
       )
@@
         )
         (path "/612afcad-8da9-4dff-bf3c-8828929809ff/8ccdbec3-7661-4a0b-9858-5169c364aebb"
-          (reference "TP3") (unit 1)
+          (reference "TP11") (unit 1)
         )
         (path "/612afcad-8da9-4dff-bf3c-8828929809ff/0c4bd054-86d6-4fc6-b8bd-5dc40d9d4357"
-          (reference "TP7") (unit 1)
+          (reference "TP14") (unit 1)
         )
         (path "/612afcad-8da9-4dff-bf3c-8828929809ff/853a01c4-0f0d-42ee-a9e8-050403071668"
-          (reference "TP16") (unit 1)
+          (reference "TP22") (unit 1)
         )
       )
@@
     (instances
       (project "magnetotorqer-drive-board"
-        (path "/612afcad-8da9-4dff-bf3c-8828929809ff/8ccdbec3-7661-4a0b-9858-5169c364aebb" (page "11"))
-        (path "/612afcad-8da9-4dff-bf3c-8828929809ff/0c4bd054-86d6-4fc6-b8bd-5dc40d9d4357" (page "9"))
-        (path "/612afcad-8da9-4dff-bf3c-8828929809ff/853a01c4-0f0d-42ee-a9e8-050403071668" (page "15"))
+        (path "/612afcad-8da9-4dff-bf3c-8828929809ff/8ccdbec3-7661-4a0b-9858-5169c364aebb" (page "401"))
+        (path "/612afcad-8da9-4dff-bf3c-8828929809ff/0c4bd054-86d6-4fc6-b8bd-5dc40d9d4357" (page "501"))
+        (path "/612afcad-8da9-4dff-bf3c-8828929809ff/853a01c4-0f0d-42ee-a9e8-050403071668" (page "601"))
       )
     )
@@
       (project "magnetotorqer-drive-board"
         (path "/612afcad-8da9-4dff-bf3c-8828929809ff" (page "7"))
-        (path "/612afcad-8da9-4dff-bf3c-8828929809ff/8ccdbec3-7661-4a0b-9858-5169c364aebb" (page "7"))
-        (path "/612afcad-8da9-4dff-bf3c-8828929809ff/0c4bd054-86d6-4fc6-b8bd-5dc40d9d4357" (page "8"))
-        (path "/612afcad-8da9-4dff-bf3c-8828929809ff/853a01c4-0f0d-42ee-a9e8-050403071668" (page "12"))
+        (path "/612afcad-8da9-4dff-bf3c-8828929809ff/8ccdbec3-7661-4a0b-9858-5169c364aebb" (page "4037"))
+        (path "/612afcad-8da9-4dff-bf3c-8828929809ff/0c4bd054-86d6-4fc6-b8bd-5dc40d9d4357" (page "503"))
+        (path "/612afcad-8da9-4dff-bf3c-8828929809ff/853a01c4-0f0d-42ee-a9e8-050403071668" (page "603"))
       )
     )
@@
     (instances
       (project "magnetotorqer-drive-board"
-        (path "/612afcad-8da9-4dff-bf3c-8828929809ff/8ccdbec3-7661-4a0b-9858-5169c364aebb" (page "13"))
-        (path "/612afcad-8da9-4dff-bf3c-8828929809ff/0c4bd054-86d6-4fc6-b8bd-5dc40d9d4357" (page "5"))
-        (path "/612afcad-8da9-4dff-bf3c-8828929809ff/853a01c4-0f0d-42ee-a9e8-050403071668" (page "14"))
-      )
-    )
+        (path "/612afcad-8da9-4dff-bf3c-8828929809ff/8ccdbec3-7661-4a0b-9858-5169c364aebb" (page "402"))
+        (path "/612afcad-8da9-4dff-bf3c-8828929809ff/0c4bd054-86d6-4fc6-b8bd-5dc40d9d4357" (page "502"))
+        (path "/612afcad-8da9-4dff-bf3c-8828929809ff/853a01c4-0f0d-42ee-a9e8-050403071668" (page "602"))
+      )
+    )
