File: revA/h_bridge.kicad_sch (KiCad schematic)
At the start: 6 parts, among them U6 DRV8838DSGT

Commit message: working
Parts:
- C22: footprint Capacitor_SMD:C_0402_1005Metric -> Capacitor_SMD:C_0603_1608Metric
- R19, R20, R21, R22: footprint Resistor_SMD:R_0402_1005Metric -> Resistor_SMD:R_0603_1608Metric

Commit message: placement
Connections:
- net +3V3 renamed +3V3D
Changed lines of the file:
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@@
+      (effects (font (size 1.27 1.27)) hide)
+    )
+    (property "Manufacturer" "" (at 167.64 127 0)
+      (effects (font (size 1.27 1.27)) hide)
+    )
+    (property "Mfr. Part No" "" (at 167.64 127 0)
+      (effects (font (size 1.27 1.27)) hide)
+    )
+    (property "Description" "" (at 167.64 127 0)
       (effects (font (size 1.27 1.27)) hide)
     )

Commit message: working
Parts:
- C22: Manufacturer TDK -> (none); Mfr. Part No CGA2B3X7R1H104K050BE -> (none)
Other:
- title: (none) -> SCHEMATIC, CUBESAT MAGNETORQER DRIVER

Commit message: worked review changes
Parts:
- C?: renamed from C22; Manufacturer (none) -> TDK Corporation; Mfr. Part No (none) -> CGA3E2X7R1H104K080AE; Value2 (none) -> 50V
- R?: renamed from R22; Manufacturer (none) -> Stackpole Electronics Inc; Mfr. Part No (none) -> RMCF0603FG1K00; Value2 (none) -> 100mW
- R?: renamed from R20; Manufacturer (none) -> Stackpole Electronics Inc; Mfr. Part No (none) -> RMCF0603FG1K00; Value2 (none) -> 100mW
- R?: renamed from R19; Manufacturer (none) -> Stackpole Electronics Inc; Mfr. Part No (none) -> RMCF0603FG1K00; Value2 (none) -> 100mW
- R?: renamed from R21; Manufacturer (none) -> Stackpole Electronics Inc; Mfr. Part No (none) -> RMCF0603FT100K; Value2 (none) -> 100mW
- U?: renamed from U6; value DRV8838DSGT -> DRV8838; symbol magnetotorquer-test-board:DRV8838DSGT -> SierraLobo:DRV8838DSGT; Manufacturer (none) -> Texas Instruments; Mfr. Part No (none) -> DRV8838DSGT
