File: revA/i_fb.kicad_sch (KiCad schematic)
At the start: 8 parts, among them U7 INA199A2xDCK

Commit message: exported init pdf
Parts:
- renumbered TP3 to TP1, TP4 to TP2, TP1 to TP3, TP2 to TP4
Changed lines of the file:
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@@
   (symbol (lib_id "Connector:TestPoint") (at 278.13 154.94 0) (unit 1)
     (in_bom no) (on_board yes) (dnp no) (fields_autoplaced)
-    (property "Reference" "TP3" (at 280.67 151.003 0)
+    (property "Reference" "TP1" (at 280.67 151.003 0)
       (effects (font (size 1.27 1.27)) (justify left))
     )
@@
   (symbol (lib_id "SierraLobo:+1V65A") (at 190.5 144.78 0) (unit 1)
     (in_bom yes) (on_board yes) (dnp no) (fields_autoplaced)
-    (property "Reference" "#PWR0103" (at 190.5 148.59 0)
+    (property "Reference" "#PWR084" (at 190.5 148.59 0)
       (effects (font (size 1.27 1.27)) hide)
     )
@@
   (symbol (lib_id "Connector:TestPoint") (at 278.13 176.53 0) (unit 1)
     (in_bom yes) (on_board yes) (dnp no)
-    (property "Reference" "TP2" (at 280.67 172.593 0)
+    (property "Reference" "TP4" (at 280.67 172.593 0)
       (effects (font (size 1.27 1.27)) (justify left))
     )
@@
   (symbol (lib_id "Connector:TestPoint") (at 278.13 162.56 0) (unit 1)
     (in_bom no) (on_board yes) (dnp no) (fields_autoplaced)
-    (property "Reference" "TP4" (at 280.67 158.623 0)
+    (property "Reference" "TP2" (at 280.67 158.623 0)
       (effects (font (size 1.27 1.27)) (justify left))
     )
@@
   (symbol (lib_id "Connector:TestPoint") (at 278.13 170.18 0) (unit 1)
     (in_bom yes) (on_board yes) (dnp no)
-    (property "Reference" "TP1" (at 280.67 166.243 0)
-      (effects (font (size 1.27 1.27)) (justify left))
-    )
+    (property "Reference" "TP3" (at 280.67 166.243 0)
+      (effects (font (size 1.27 1.27)) (justify left))
+    )

Commit message: working
Parts:
- removed TP1, TP2: 2mm Pad, TestPoint:TestPoint_Pad_D2.0mm, symbol Connector:TestPoint
- removed TP3, TP4: ${NET_NAME(1)}, TestPoint:TestPoint_Keystone_5000-5004_Miniature, symbol Connector:TestPoint
- C23, C24: footprint Capacitor_SMD:C_0402_1005Metric -> Capacitor_SMD:C_0603_1608Metric
Other:
- note removed: "TEST POINTS"

Commit message: working
Parts:
- C24: now fitted
Changed lines of the file:
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@@
   )
   (symbol (lib_id "Device:C") (at 190.5 149.86 0) (mirror y) (unit 1)
-    (in_bom yes) (on_board yes) (dnp yes)
+    (in_bom yes) (on_board yes) (dnp no)
     (property "Reference" "C24" (at 187.579 148.9515 0)
       (effects (font (size 1.27 1.27)) (justify left))

Commit message: placement
Connections:
- net +3V3 renamed +1V65A
- net VCC renamed +3V3A
Changed lines of the file:
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@@
-    (stroke (width 0) (type default))
-  )
-  (wire (pts (xy 177.8 104.14) (xy 181.61 104.14))
     (stroke (width 0) (type default))
   )
@@
   (hierarchical_label "V_SENSE" (shape output) (at 234.95 132.08 0) (fields_autoplaced)
     (effects (font (size 1.27 1.27)) (justify left))
-  )
-  (hierarchical_label "VCC" (shape input) (at 177.8 104.14 180) (fields_autoplaced)
-    (effects (font (size 1.27 1.27)) (justify right))
   )
   (hierarchical_label "IN-" (shape input) (at 177.8 134.62 180) (fields_autoplaced)
@@
     )
   )
+  (symbol (lib_id "SierraLobo:+3V3A") (at 181.61 104.14 0) (unit 1)
+    (in_bom yes) (on_board yes) (dnp no) (fields_autoplaced)
+    (property "Reference" "#PWR019" (at 181.61 107.95 0)
+      (effects (font (size 1.27 1.27)) hide)
+    )
+    (property "Value" "+3V3A" (at 181.61 100.33 0)
+      (effects (font (size 1.27 1.27)))
+    )
+    (property "Footprint" "" (at 181.61 104.14 0)
+      (effects (font (size 1.27 1.27)) hide)
+    )
+    (property "Datasheet" "" (at 181.61 104.14 0)
+      (effects (font (size 1.27 1.27)) hide)
+    )
+    (property "Manufacturer" "" (at 181.61 104.14 0)
+      (effects (font (size 1.27 1.27)) hide)
+    )
+    (property "Mfr. Part No" "" (at 181.61 104.14 0)
+      (effects (font (size 1.27 1.27)) hide)
+    )
+    (property "Description" "" (at 181.61 104.14 0)
+      (effects (font (size 1.27 1.27)) hide)
+    )
+    (pin "1")
+    (instances
+      (project "magnetotorqer-drive-board"
+        (path "/612afcad-8da9-4dff-bf3c-8828929809ff"
+          (reference "#PWR019") (unit 1)
+        )
+        (path "/612afcad-8da9-4dff-bf3c-8828929809ff/8ccdbec3-7661-4a0b-9858-5169c364aebb/765443f8-c18e-4cd2-97d5-a5c0f8a3785d"
+          (reference "#PWR0191") (unit 1)
+        )
+        (path "/612afcad-8da9-4dff-bf3c-8828929809ff/0c4bd054-86d6-4fc6-b8bd-5dc40d9d4357/765443f8-c18e-4cd2-97d5-a5c0f8a3785d"
+          (reference "#PWR0192") (unit 1)
+        )
+        (path "/612afcad-8da9-4dff-bf3c-8828929809ff/853a01c4-0f0d-42ee-a9e8-050403071668/765443f8-c18e-4cd2-97d5-a5c0f8a3785d"
+          (reference "#PWR0193") (unit 1)
+        )
+      )
+    )
+  )
   (symbol (lib_id "Device:C") (at 190.5 149.86 0) (mirror y) (unit 1)
     (in_bom yes) (on_board yes) (dnp no)
@@
       (effects (font (size 1.27 1.27)) hide)
     )
+    (property "Manufacturer" "" (at 190.5 144.78 0)
+      (effects (font (size 1.27 1.27)) hide)
+    )
+    (property "Mfr. Part No" "" (at 190.5 144.78 0)
+      (effects (font (size 1.27 1.27)) hide)
+    )
+    (property "Description" "" (at 190.5 144.78 0)
+      (effects (font (size 1.27 1.27)) hide)
+    )

Commit message: working
Parts:
- C24: Manufacturer TDK -> (none); Mfr. Part No CGA2B3X7R1H104K050BE -> (none)
Other:
- title: Current Sense Amplifier -> SCHEMATIC, CUBESAT MAGNETORQER DRIVER
Changed lines of the file:
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@@
   (paper "B")
   (title_block
-    (title "Current Sense Amplifier")
-    (date "2023-06-23")
+    (title "SCHEMATIC, CUBESAT MAGNETORQER DRIVER")
+    (date "2023-06-28")
     (rev "A")
     (comment 1 "CH")
     (comment 2 "CH")
+    (comment 3 "RD21-6005")
   )
   (junction (at 190.5 144.78) (diameter 0) (color 0 0 0 0)
@@
         )
         (path "/612afcad-8da9-4dff-bf3c-8828929809ff/8ccdbec3-7661-4a0b-9858-5169c364aebb/765443f8-c18e-4cd2-97d5-a5c0f8a3785d"
-          (reference "#PWR0191") (unit 1)
-        )
-        (path "/612afcad-8da9-4dff-bf3c-8828929809ff/0c4bd054-86d6-4fc6-b8bd-5dc40d9d4357/765443f8-c18e-4cd2-97d5-a5c0f8a3785d"
-          (reference "#PWR0192") (unit 1)
-        )
-        (path "/612afcad-8da9-4dff-bf3c-8828929809ff/853a01c4-0f0d-42ee-a9e8-050403071668/765443f8-c18e-4cd2-97d5-a5c0f8a3785d"
-          (reference "#PWR0193") (unit 1)
+          (reference "#PWR075") (unit 1)
+        )
+        (path "/612afcad-8da9-4dff-bf3c-8828929809ff/0c4bd054-86d6-4fc6-b8bd-5dc40d9d4357/765443f8-c18e-4cd2-97d5-a5c0f8a3785d"
+          (reference "#PWR080") (unit 1)
+        )
+        (path "/612afcad-8da9-4dff-bf3c-8828929809ff/853a01c4-0f0d-42ee-a9e8-050403071668/765443f8-c18e-4cd2-97d5-a5c0f8a3785d"
+          (reference "#PWR0125") (unit 1)
         )
       )
@@
       (effects (font (size 1.27 1.27)) hide)
     )
-    (property "Description" "CAP CER 0.1UF 50V X7R 0402" (at 190.5 149.86 0)
-      (effects (font (size 1.27 1.27)) hide)
-    )
-    (property "Manufacturer" "TDK" (at 190.5 149.86 0)
-      (effects (font (size 1.27 1.27)) hide)
-    )
-    (property "Mfr. Part No" "CGA2B3X7R1H104K050BE" (at 190.5 149.86 0)
+    (property "Description" "" (at 190.5 149.86 0)
+      (effects (font (size 1.27 1.27)) hide)
+    )
+    (property "Manufacturer" "" (at 190.5 149.86 0)
+      (effects (font (size 1.27 1.27)) hide)
+    )
+    (property "Mfr. Part No" "" (at 190.5 149.86 0)
       (effects (font (size 1.27 1.27)) hide)
     )
@@
         )
         (path "/612afcad-8da9-4dff-bf3c-8828929809ff/8ccdbec3-7661-4a0b-9858-5169c364aebb/765443f8-c18e-4cd2-97d5-a5c0f8a3785d"
-          (reference "C29") (unit 1)
-        )
-        (path "/612afcad-8da9-4dff-bf3c-8828929809ff/0c4bd054-86d6-4fc6-b8bd-5dc40d9d4357/765443f8-c18e-4cd2-97d5-a5c0f8a3785d"
-          (reference "C32") (unit 1)
-        )
-        (path "/612afcad-8da9-4dff-bf3c-8828929809ff/853a01c4-0f0d-42ee-a9e8-050403071668/765443f8-c18e-4cd2-97d5-a5c0f8a3785d"
-          (reference "C55") (unit 1)
+          (reference "C30") (unit 1)
+        )
+        (path "/612afcad-8da9-4dff-bf3c-8828929809ff/0c4bd054-86d6-4fc6-b8bd-5dc40d9d4357/765443f8-c18e-4cd2-97d5-a5c0f8a3785d"
+          (reference "C33") (unit 1)
+        )
+        (path "/612afcad-8da9-4dff-bf3c-8828929809ff/853a01c4-0f0d-42ee-a9e8-050403071668/765443f8-c18e-4cd2-97d5-a5c0f8a3785d"
+          (reference "C56") (unit 1)
         )
       )
@@
         )
         (path "/612afcad-8da9-4dff-bf3c-8828929809ff/0c4bd054-86d6-4fc6-b8bd-5dc40d9d4357/765443f8-c18e-4cd2-97d5-a5c0f8a3785d"
-          (reference "#PWR081") (unit 1)
-        )
-        (path "/612afcad-8da9-4dff-bf3c-8828929809ff/853a01c4-0f0d-42ee-a9e8-050403071668/765443f8-c18e-4cd2-97d5-a5c0f8a3785d"
-          (reference "#PWR0124") (unit 1)
+          (reference "#PWR082") (unit 1)
+        )
+        (path "/612afcad-8da9-4dff-bf3c-8828929809ff/853a01c4-0f0d-42ee-a9e8-050403071668/765443f8-c18e-4cd2-97d5-a5c0f8a3785d"
+          (reference "#PWR0127") (unit 1)
         )
       )
@@
         )
         (path "/612afcad-8da9-4dff-bf3c-8828929809ff/0c4bd054-86d6-4fc6-b8bd-5dc40d9d4357/765443f8-c18e-4cd2-97d5-a5c0f8a3785d"
-          (reference "#PWR083") (unit 1)
-        )
-        (path "/612afcad-8da9-4dff-bf3c-8828929809ff/853a01c4-0f0d-42ee-a9e8-050403071668/765443f8-c18e-4cd2-97d5-a5c0f8a3785d"
-          (reference "#PWR0126") (unit 1)
+          (reference "#PWR084") (unit 1)
+        )
+        (path "/612afcad-8da9-4dff-bf3c-8828929809ff/853a01c4-0f0d-42ee-a9e8-050403071668/765443f8-c18e-4cd2-97d5-a5c0f8a3785d"
+          (reference "#PWR0129") (unit 1)
         )
       )
@@
         )
         (path "/612afcad-8da9-4dff-bf3c-8828929809ff/0c4bd054-86d6-4fc6-b8bd-5dc40d9d4357/765443f8-c18e-4cd2-97d5-a5c0f8a3785d"
-          (reference "#PWR080") (unit 1)
-        )
-        (path "/612afcad-8da9-4dff-bf3c-8828929809ff/853a01c4-0f0d-42ee-a9e8-050403071668/765443f8-c18e-4cd2-97d5-a5c0f8a3785d"
-          (reference "#PWR0123") (unit 1)
+          (reference "#PWR081") (unit 1)
+        )
+        (path "/612afcad-8da9-4dff-bf3c-8828929809ff/853a01c4-0f0d-42ee-a9e8-050403071668/765443f8-c18e-4cd2-97d5-a5c0f8a3785d"
+          (reference "#PWR0126") (unit 1)
         )
       )
@@
         )
         (path "/612afcad-8da9-4dff-bf3c-8828929809ff/0c4bd054-86d6-4fc6-b8bd-5dc40d9d4357/765443f8-c18e-4cd2-97d5-a5c0f8a3785d"
-          (reference "#PWR082") (unit 1)
-        )
-        (path "/612afcad-8da9-4dff-bf3c-8828929809ff/853a01c4-0f0d-42ee-a9e8-050403071668/765443f8-c18e-4cd2-97d5-a5c0f8a3785d"
-          (reference "#PWR0125") (unit 1)
+          (reference "#PWR083") (unit 1)
+        )
+        (path "/612afcad-8da9-4dff-bf3c-8828929809ff/853a01c4-0f0d-42ee-a9e8-050403071668/765443f8-c18e-4cd2-97d5-a5c0f8a3785d"
+          (reference "#PWR0128") (unit 1)
         )
       )
@@
       (effects (font (size 1.27 1.27)) hide)
     )
-    (property "Description" "CAP CER 0.1UF 50V X7R 0402" (at 194.31 109.22 0)
-      (effects (font (size 1.27 1.27)) hide)
-    )
-    (property "Manufacturer" "TDK" (at 194.31 109.22 0)
-      (effects (font (size 1.27 1.27)) hide)
-    )
-    (property "Mfr. Part No" "CGA2B3X7R1H104K050BE" (at 194.31 109.22 0)
+    (property "Description" "" (at 194.31 109.22 0)
+      (effects (font (size 1.27 1.27)) hide)
+    )
+    (property "Manufacturer" "" (at 194.31 109.22 0)
+      (effects (font (size 1.27 1.27)) hide)
+    )
+    (property "Mfr. Part No" "" (at 194.31 109.22 0)
       (effects (font (size 1.27 1.27)) hide)
     )
@@
         )
         (path "/612afcad-8da9-4dff-bf3c-8828929809ff/8ccdbec3-7661-4a0b-9858-5169c364aebb/765443f8-c18e-4cd2-97d5-a5c0f8a3785d"
-          (reference "C30") (unit 1)
-        )
-        (path "/612afcad-8da9-4dff-bf3c-8828929809ff/0c4bd054-86d6-4fc6-b8bd-5dc40d9d4357/765443f8-c18e-4cd2-97d5-a5c0f8a3785d"
-          (reference "C33") (unit 1)
-        )
-        (path "/612afcad-8da9-4dff-bf3c-8828929809ff/853a01c4-0f0d-42ee-a9e8-050403071668/765443f8-c18e-4cd2-97d5-a5c0f8a3785d"
-          (reference "C56") (unit 1)
-        )
-      )
+          (reference "C29") (unit 1)
+        )
+        (path "/612afcad-8da9-4dff-bf3c-8828929809ff/0c4bd054-86d6-4fc6-b8bd-5dc40d9d4357/765443f8-c18e-4cd2-97d5-a5c0f8a3785d"
+          (reference "C32") (unit 1)
+        )
+        (path "/612afcad-8da9-4dff-bf3c-8828929809ff/853a01c4-0f0d-42ee-a9e8-050403071668/765443f8-c18e-4cd2-97d5-a5c0f8a3785d"
+          (reference "C55") (unit 1)
+        )
+      )

Commit message: worked review changes
Parts:
- removed C23: 0.01uF, Capacitor_SMD:C_0603_1608Metric, symbol Device:C
- C? (x2): renamed from C24; Manufacturer (none) -> TDK Corporation; Mfr. Part No (none) -> CGA3E2X7R1H104K080AE; Value2 (none) -> 50V
- U?: renamed from U7; value INA199A2xDCK -> INA199A2; Manufacturer (none) -> Texas Instruments; Mfr. Part No (none) -> INA199A2DCKT
