File: revA/magnetotorqer-drive-board.kicad_sch (KiCad schematic)
At the start: 41 parts, among them J3 Conn_01x02, J4 Conn_01x02, J5 Conn_01x02, J6 Conn_01x02, J7 Conn_01x02, J8 Conn_01x02, P1 Card Edge for HSEC8-160-01-S-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, Q1 BSZ180, Q2 BSZ180, Q3 MMBT4401WT1G, U1 SN74LVC2G17DBVR, U3 MCP1700T-33, U4 ATL431BQ

Commit message: working
Parts:
- removed C6: 0.1uF, Capacitor_SMD:C_0603_1608Metric, symbol Device:C
- removed C7 (x2): 47uF, Capacitor_Tantalum_SMD:CP_EIA-7343-43_Kemet-X, symbol Device:C_Polarized_US
- removed Q1, Q2: BSZ180, SierraLobo:PG-TSDSON-8_3.3x3.3mm, symbol SierraLobo:BSZ086
- removed Q3: MMBT4401WT1G, Package_TO_SOT_SMD:SOT-323_SC-70, symbol Device:Q_NPN_BEC
- removed R23, R40: 300mR, Resistor_SMD:R_0805_2012Metric, symbol Device:R_US
- removed R41: ?, Resistor_SMD:R_0805_2012Metric, symbol Device:R_US
- removed R6: 100k, Resistor_SMD:R_0603_1608Metric, symbol Device:R_US
- added C101: 0.1uF, Capacitor_SMD:C_0603_1608Metric, symbol Device:C
- added C102, C103: 1uF, Capacitor_SMD:C_0603_1608Metric, symbol Device:C
- added C7 (x2): 47uF, Capacitor_Tantalum_SMD:CP_EIA-7343-43_Kemet-X, symbol Device:C_Polarized_US
- added NTC1, NTC2, NTC3: 10k, symbol Device:Thermistor_NTC_US
- added Q4, Q5: BSZ180, SierraLobo:PG-TSDSON-8_3.3x3.3mm, symbol SierraLobo:BSZ086
- added Q6: MMBT4401WT1G, Package_TO_SOT_SMD:SOT-323_SC-70, symbol Device:Q_NPN_BEC
- added R114, R120: 100k, Resistor_SMD:R_0603_1608Metric, symbol Device:R_US
- added R115, R119: 1k, Resistor_SMD:R_0603_1608Metric, symbol Device:R_US
- added U23: MCP1700T-50, Package_TO_SOT_SMD:SOT-89-3, symbol Regulator_Linear:MCP1700x-330xxMB
- R3: value 100k -> 10k; footprint Resistor_SMD:R_0603_1608Metric -> (none)
- R4, R5: value 1k -> 10k; footprint Resistor_SMD:R_0603_1608Metric -> (none)
Connections:
- net 1V65A is gone; now on net +3V3: C19.1, R12.2, R13.1, U4.2 (K)
- net 3V3A is gone; now on net +3V3: C17.1, U3.3 (VO)
- net +3V3: now also R3.1, R4.1, R5.1
- net 5V_SYS: no longer R3.1
- net GND: now also C102.2, C103.2, C7.2, C7.2, NTC1.2, NTC2.2, NTC3.2, Q6.2 (E), U23.1 (GND)
- net MTDB_PWR_EN: now also R120.1
- net X_TEMP: now also R3.2, NTC1.1
- net Y_TEMP: now also R4.2, NTC2.1
- net Z_TEMP: now also R5.2, NTC3.1
- net 5V renamed VAA
- net VAA: now also C102.1, C7.1, C7.1, Q4.5 (D), Q5.5 (D), U23.2 (VI)
- new net: Q6.1 (B), R120.2
- new net: C101.2, Q6.3 (C), R114.2, R115.2, R119.2
- new net: Q5.4 (G), R115.1
- new net: Q4.4 (G), R119.1
- new net +5VA: C103.1, U23.3 (VO)
- new net VBATT: C101.1, Q4.1 (S), Q5.1 (S), R114.1
Other:
- sheet X Driver ports: added DIN, REG_EN, SCK, VIN, V_RSEN, ~{SYNC}; removed 1V65A, 3V3A, 3V3D, 5VA, DRV_IN, ISENSE, SENSE, ~{AMP_SHDN}
- sheet Y Driver ports: added DIN, REG_EN, SCK, VIN, V_RSEN, ~{SYNC}; removed 1V65A, 3V3A, 3V3D, 5VA, DRV_IN, ISENSE, SENSE, ~{AMP_SHDN}
- sheet Z Driver ports: added DIN, REG_EN, SCK, VIN, V_RSEN, ~{SYNC}; removed 1V65A, 3V3A, 3V3D, 5VA, DRV_IN, ISENSE, SENSE, ~{AMP_SHDN}
- note added: "250mA MAX"
- note added: "5V ANALOG"
- note added: "Attached to MTQs"
- note added: "MTQ CONTROLLER"
- note added: "MTQ DRIVERs"
- note added: "NTC BIAS"
- note added: "power cycle capability to 5VA, 3VA?"
- note removed: "MTQ CONTROL"
- note removed: "MTQ DRIVERS"
- moved on the sheet: C1, C16, C17, C18, C19, C2, C3, C4, H1, H2, H3, H4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

Commit message: exported init pdf
Parts:
- added C6, C7: 1uF, Capacitor_SMD:C_0603_1608Metric, symbol Device:C
- added U2: MCP1700T-33, Package_TO_SOT_SMD:SOT-89-3, symbol Regulator_Linear:MCP1700x-330xxMB
Connections:
- net GND: now also C6.2, C7.2, U2.1 (GND)
- net VAA: now also C6.1, U2.2 (VI)
- net 5V_SYS: no longer names the net of P1.59 (Pin_59)
- net 5V_SYS: no longer P1.60 (Pin_60)
- new net: C7.1, U2.3 (VO)
- no-connect marks 108 -> 110
Other:
- removed sheet 3V3 Digital Regulator
- note added: "power cycle capability to these regs?"
- note removed: "3V3 REGULATOR"
- note removed: "MTQ TEMP SENSOR BIAS"
- note removed: "POWER"
- note removed: "power cycle capability to 5VA, 3VA?"
- moved on the sheet: C7

Commit message: working
Parts:
- removed C101: 0.1uF, Capacitor_SMD:C_0603_1608Metric, symbol Device:C
- removed C102, C103, C16, C17, C18: 1uF, Capacitor_SMD:C_0603_1608Metric, symbol Device:C
- removed C19: 10uF, Capacitor_SMD:C_0805_2012Metric, symbol Device:C
- removed C7 (x2): 47uF, Capacitor_Tantalum_SMD:CP_EIA-7343-43_Kemet-X, symbol Device:C_Polarized_US
- removed Q4, Q5: BSZ180, SierraLobo:PG-TSDSON-8_3.3x3.3mm, symbol SierraLobo:BSZ086
- removed Q6: MMBT4401WT1G, Package_TO_SOT_SMD:SOT-323_SC-70, symbol Device:Q_NPN_BEC
- removed R114, R120: 100k, Resistor_SMD:R_0603_1608Metric, symbol Device:R_US
- removed R115, R119: 1k, Resistor_SMD:R_0603_1608Metric, symbol Device:R_US
- removed R12: 10k, Resistor_SMD:R_0603_1608Metric, symbol Device:R_US
- removed R13: 12.4k, Resistor_SMD:R_0603_1608Metric, symbol Device:R_US
- removed R14: 4.1k, Resistor_SMD:R_0603_1608Metric, symbol Device:R_US
- removed U1: SN74LVC2G17DBVR, Package_TO_SOT_SMD:SOT-23-6, symbol SierraLobo:SN74LVC2G17DBVR
- removed U2, U3: MCP1700T-33, Package_TO_SOT_SMD:SOT-89-3, symbol Regulator_Linear:MCP1700x-330xxMB
- removed U23: MCP1700T-50, Package_TO_SOT_SMD:SOT-89-3, symbol Regulator_Linear:MCP1700x-330xxMB
- removed U4: ATL431BQ, Package_TO_SOT_SMD:SOT-23, symbol SierraLobo:TLVH431BQxDBV
- added C10, C9: 0.1uF, Capacitor_SMD:C_0603_1608Metric, symbol Device:C
- added C8: 1uF, Capacitor_SMD:C_0805_2012Metric, symbol Device:C
- added D1, D2: ESD321DPYR, SierraLobo:D_0402_1005Metric, symbol Device:D_Zener
- added J1: ZX62-AB-5PA(31), SierraLobo:ZX62-AB-5PA(31), symbol Connector:USB_B_Micro
- added R3, R4: 220, Resistor_SMD:R_0603_1608Metric, symbol Device:R_US
- added U1, U2: 74LVC1G17, Package_TO_SOT_SMD:SOT-353_SC-70-5, symbol SierraLobo:74LVC1G17
- added U3, U4: MCP9700AT-E/LT, Package_TO_SOT_SMD:SOT-353_SC-70-5, symbol Sensor_Temperature:MCP9700Ax-ELT
- C5: footprint (none) -> Capacitor_SMD:C_0603_1608Metric
- C6: value 1uF -> 0.1uF
- C7: footprint Capacitor_SMD:C_0603_1608Metric -> Capacitor_SMD:C_0805_2012Metric; Manufacturer (none) -> TDK; Mfr. Part No (none) -> CGA3E1X7R1V105K080AE
- J2: renamed from J4; value Conn_01x02 -> T1M-02-F-SH-L; footprint SierraLobo:SAMTEC_T1M-02-F-SV-L-P -> SierraLobo:SAMTEC_T1M-02-F-SH-L-K; Mfr. Part No T1M-02-F-SV-L-P -> T1M-02-F-SH-L-K
- J3: renamed from J5; value Conn_01x02 -> T1M-02-F-SH-L; footprint SierraLobo:SAMTEC_T1M-02-F-SV-L-P -> SierraLobo:SAMTEC_T1M-02-F-SH-L-K; Mfr. Part No T1M-02-F-SV-L-P -> T1M-02-F-SH-L-K
- J4: renamed from J3; value Conn_01x02 -> T1M-02-F-SH-L; footprint SierraLobo:SAMTEC_T1M-02-F-SV-L-P -> SierraLobo:SAMTEC_T1M-02-F-SH-L-K; Mfr. Part No T1M-02-F-SV-L-P -> T1M-02-F-SH-L-K
- J5: renamed from J6; value Conn_01x02 -> T1M-02-F-SH-L; footprint SierraLobo:SAMTEC_T1M-02-F-SV-L-P -> SierraLobo:SAMTEC_T1M-02-F-SH-L-K; Mfr. Part No T1M-02-F-SV-L-P -> T1M-02-F-SH-L-K
- J6: renamed from J7; value Conn_01x02 -> T1M-02-F-SH-L; footprint SierraLobo:SAMTEC_T1M-02-F-SV-L-P -> SierraLobo:SAMTEC_T1M-02-F-SH-L-K; Mfr. Part No T1M-02-F-SV-L-P -> T1M-02-F-SH-L-K
- J7: renamed from J8; value Conn_01x02 -> T1M-02-F-SH-L; footprint SierraLobo:SAMTEC_T1M-02-F-SV-L-P -> SierraLobo:SAMTEC_T1M-02-F-SH-L-K; Mfr. Part No T1M-02-F-SV-L-P -> T1M-02-F-SH-L-K
- R1, R2: footprint (none) -> Resistor_SMD:R_0603_1608Metric
- R5: renamed from R3; footprint (none) -> Resistor_SMD:R_0603_1608Metric
- R6: renamed from R4; footprint (none) -> Resistor_SMD:R_0603_1608Metric
- R7: renamed from R5; footprint (none) -> Resistor_SMD:R_0603_1608Metric
Connections:
- net +3V3: now also C6.1, R3.1, R4.1, U1.5 (VCC), U2.5 (VCC)
- net GND: now also C10.2, C8.2, C9.2, D1.2 (A), D2.2 (A), J1.5 (GND), J1.6 (Shield), U1.3 (GND), U2.3 (GND), U3.2 (GND), U4.2 (GND)
- net RX_4: now also P1.41 (Pin_41), U2.4
- net RX_MCU: now also U1.4
- net TX_4: now also P1.42 (Pin_42)
- net VAA: no longer C6.1
- net VBATT: now also P1.100 (Pin_100), P1.97 (Pin_97), P1.98 (Pin_98), P1.99 (Pin_99)
- net at C7.1: now also R3.2, U3.4 (V_{DD})
- net at R1.2: now also U1.2
- net at R2.2: now also U2.2
- net LED_VCC: now reaches P1.15 (Pin_15)
- net ~{FAULT}: now reaches P1.43 (Pin_43)
- net PWR_EN: now reaches P1.44 (Pin_44)
- new net: C8.1, R4.2, U4.4 (V_{DD})
- new net 5V_USB: J1.1 (VBUS)
- new net D+: D2.1 (K), J1.3 (D+)
- new net D-: D1.1 (K), J1.2 (D-)
- new net TEMP_A: C9.1, U3.3 (V_{OUT})
- new net TEMP_B: C10.1, U4.3 (V_{OUT})
- no-connect marks 110 -> 109
Other:
- added sheet Power (power.kicad_sch)
- sheet Control ports: added AIN0, AIN1, AIN2, AIN3, AIN4, AIN5, AIN6, HARD_RST, MISO, MOSI, PA12, PA13, PA14, PA15, PA16, PA20, PB00, PB01, PB02, PB03, PB04, PB05, PB06, PB07, PB12, PB13, PB14, PB15, PB30, PB31, RX, SCK, TX, USB_D+, USB_D-, ~{FAULT}, ~{RST}; removed none
- note added: "POWER"
- note added: "TEMP SENSORS"
- note added: "USB Connector"
- note removed: "1V65 REF"
- note removed: "250mA MAX"
- note removed: "3V3 ANALOG"
- note removed: "5V ANALOG"
- note removed: "BULK"
- note removed: "POWER SWITCH"
- note removed: "power cycle capability to these regs?"
- moved on the sheet: C1, C2, C3, C4, C5, H1, H2, H3, H4, J2, J3, J4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

Commit message: working
Parts:
- NTC1, NTC2, NTC3: Manufacturer (none) -> TE; Mfr. Part No (none) -> GA10K3A1AM; Value2 (none) -> 3976K
- P1: footprint SLI-Backplane-Blank-Card-KiCad:HSEC8-160-CARD-EDGE -> SierraLobo:HSEC8-160-CARD-EDGE; symbol payload-interface-board:Conn_02x60_Top_Bottom -> SierraLobo:EdgeConnector_HSEC8-160-01-S-DV-A-K-TR
Other:
- note added: "-40-125degC operational V_{OUT}=10mV/degC, 500mV offset 6uA quiesent"
- moved on the sheet: C10, C9

Commit message: placement
Connections:
- net RX_MCU is gone; now on net RX: U1.4
- net TX_MCU is gone; now on net TX: R2.1
- net +3V3 renamed +3V3A
- net +3V3A: no longer C5.1, C6.1, U1.5 (VCC), U2.5 (VCC)
- new net +3V3D: C5.1, C6.1, U1.5 (VCC), U2.5 (VCC)
Changed lines of the file:
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@@
     (effects (font (size 1.27 1.27)) (justify left bottom))
   )
-  (label "RX_MCU" (at 199.39 55.88 180) (fields_autoplaced)
+  (label "RX" (at 199.39 55.88 180) (fields_autoplaced)
     (effects (font (size 1.27 1.27)) (justify right bottom))
   )
@@
     (effects (font (size 1.27 1.27)) (justify right bottom))
   )
-  (label "TX_MCU" (at 199.39 87.63 180) (fields_autoplaced)
+  (label "TX" (at 199.39 87.63 180) (fields_autoplaced)
     (effects (font (size 1.27 1.27)) (justify right bottom))
   )
@@
       (effects (font (size 1.27 1.27)) hide)
     )
+    (property "Manufacturer" "" (at 269.24 193.04 0)
+      (effects (font (size 1.27 1.27)) hide)
+    )
+    (property "Mfr. Part No" "" (at 269.24 193.04 0)
+      (effects (font (size 1.27 1.27)) hide)
+    )
+    (property "Description" "" (at 269.24 193.04 0)
+      (effects (font (size 1.27 1.27)) hide)
+    )
     (pin "1")
     (instances
@@
       (effects (font (size 1.27 1.27)) hide)
     )
+    (property "Manufacturer" "" (at 135.89 34.29 0)
+      (effects (font (size 1.27 1.27)) hide)
+    )
+    (property "Mfr. Part No" "" (at 135.89 34.29 0)
+      (effects (font (size 1.27 1.27)) hide)
+    )
+    (property "Description" "" (at 135.89 34.29 0)
+      (effects (font (size 1.27 1.27)) hide)
+    )
     (pin "1")
     (instances
@@
       (effects (font (size 1.27 1.27)) hide)
     )
+    (property "Manufacturer" "" (at 185.42 66.04 0)
+      (effects (font (size 1.27 1.27)) hide)
+    )
+    (property "Mfr. Part No" "" (at 185.42 66.04 0)
+      (effects (font (size 1.27 1.27)) hide)
+    )
+    (property "Description" "" (at 185.42 66.04 0)
+      (effects (font (size 1.27 1.27)) hide)
+    )
     (pin "1")
     (instances
@@
       (effects (font (size 1.27 1.27)) hide)
     )
+    (property "Manufacturer" "" (at 355.6 171.45 0)
+      (effects (font (size 1.27 1.27)) hide)
+    )
+    (property "Mfr. Part No" "" (at 355.6 171.45 0)
+      (effects (font (size 1.27 1.27)) hide)
+    )
+    (property "Description" "" (at 355.6 171.45 0)
+      (effects (font (size 1.27 1.27)) hide)
+    )
     (pin "1")
     (instances
@@
     )
     (property "Datasheet" "" (at 393.7 171.45 0)
+      (effects (font (size 1.27 1.27)) hide)
+    )
+    (property "Manufacturer" "" (at 393.7 171.45 0)
+      (effects (font (size 1.27 1.27)) hide)
+    )
+    (property "Mfr. Part No" "" (at 393.7 171.45 0)
+      (effects (font (size 1.27 1.27)) hide)
+    )
+    (property "Description" "" (at 393.7 171.45 0)
       (effects (font (size 1.27 1.27)) hide)
     )
@@
       (effects (font (size 1.27 1.27)) hide)
     )
+    (property "Manufacturer" "" (at 269.24 165.1 0)
+      (effects (font (size 1.27 1.27)) hide)
+    )
+    (property "Mfr. Part No" "" (at 269.24 165.1 0)
+      (effects (font (size 1.27 1.27)) hide)
+    )
+    (property "Description" "" (at 269.24 165.1 0)
+      (effects (font (size 1.27 1.27)) hide)
+    )
     (pin "1")
     (instances
@@
       (effects (font (size 1.27 1.27)) hide)
     )
+    (property "Manufacturer" "" (at 374.65 171.45 0)
+      (effects (font (size 1.27 1.27)) hide)
+    )
+    (property "Mfr. Part No" "" (at 374.65 171.45 0)
+      (effects (font (size 1.27 1.27)) hide)
+    )
+    (property "Description" "" (at 374.65 171.45 0)
+      (effects (font (size 1.27 1.27)) hide)
+    )
