File: revA/power.kicad_sch (KiCad schematic)
At the start: 58 parts, among them J9 Conn_02x02_Top_Bottom, Q1 MMBT4401WT1G, Q3 BSZ180, Q3 MMDT2222A, Q4 IRLML2803, Q6 MMDT2222A, Q9 MMDT2222A, U25 AP2161W, U3 MCP1700T-50, U4 MCP1700T-33, U5 MCP1700T-33, U6 ATL431BQ

Commit message: placement
Parts:
- J9: symbol Connector_Generic:Conn_02x02_Top_Bottom -> Connector_Generic:Conn_02x02_Odd_Even
Connections:
- net +5VA: now also J9.2 (Pin_2); no longer J9.4 (Pin_4)
- net VAA: now also J9.4 (Pin_4); no longer J9.3 (Pin_3)
- net at C64.1, C8.1, J9.1 (Pin_1)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: now also J9.3 (Pin_3); no longer J9.2 (Pin_2)
- removed net +3V3: C13.1, C16.1, C17.1, R8.2, R87.1, R9.1, TP3.1, TP3.1, TP3.1, U4.3 (VO), U5.3 (VO), U6.2 (K)
- new net +1V65A: C17.1, R8.2, R9.1, TP3.1, U6.2 (K)
- new net +3V3A: C16.1, TP3.1, U5.3 (VO)
- new net +3V3D: C13.1, R87.1, TP3.1, U4.3 (VO)
Changed lines of the file:
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@@
     (stroke (width 0) (type default))
   )
-  (wire (pts (xy 182.88 215.9) (xy 193.04 215.9))
+  (wire (pts (xy 182.88 218.44) (xy 198.12 218.44))
     (stroke (width 0) (type default))
   )
@@
     (stroke (width 0) (type default))
   )
-  (wire (pts (xy 161.29 215.9) (xy 170.18 215.9))
-    (stroke (width 0) (type default))
-  )
   (wire (pts (xy 80.01 161.29) (xy 87.63 161.29))
     (stroke (width 0) (type default))
@@
     (stroke (width 0) (type default))
   )
+  (wire (pts (xy 161.29 215.9) (xy 170.18 215.9))
+    (stroke (width 0) (type default))
+  )
   (wire (pts (xy 63.5 55.88) (xy 95.25 55.88))
     (stroke (width 0) (type default))
@@
     (stroke (width 0) (type default))
   )
-  (wire (pts (xy 182.88 218.44) (xy 198.12 218.44))
+  (wire (pts (xy 182.88 215.9) (xy 194.31 215.9))
     (stroke (width 0) (type default))
   )
@@
       (effects (font (size 1.27 1.27)) hide)
     )
+    (property "Manufacturer" "" (at 351.79 170.18 0)
+      (effects (font (size 1.27 1.27)) hide)
+    )
+    (property "Mfr. Part No" "" (at 351.79 170.18 0)
+      (effects (font (size 1.27 1.27)) hide)
+    )
+    (property "Description" "" (at 351.79 170.18 0)
+      (effects (font (size 1.27 1.27)) hide)
+    )
     (pin "1")
     (instances
@@
       (effects (font (size 1.27 1.27)) hide)
     )
+    (property "Manufacturer" "" (at 309.88 175.26 0)
+      (effects (font (size 1.27 1.27)) hide)
+    )
+    (property "Mfr. Part No" "" (at 309.88 175.26 0)
+      (effects (font (size 1.27 1.27)) hide)
+    )
+    (property "Description" "" (at 309.88 175.26 0)
+      (effects (font (size 1.27 1.27)) hide)
+    )
     (pin "1")
     (instances
@@
     )
   )
-  (symbol (lib_id "Connector_Generic:Conn_02x02_Top_Bottom") (at 175.26 215.9 0) (unit 1)
+  (symbol (lib_id "Connector_Generic:Conn_02x02_Odd_Even") (at 175.26 218.44 0) (mirror x) (unit 1)
     (in_bom yes) (on_board yes) (dnp no)
-    (property "Reference" "J9" (at 176.53 209.55 0)
+    (property "Reference" "J9" (at 176.53 224.79 0)
       (effects (font (size 1.27 1.27)))
     )
-    (property "Value" "Conn_02x02_Top_Bottom" (at 176.53 212.09 0)
+    (property "Value" "Conn_02x02_Top_Bottom" (at 176.53 222.25 0)
       (effects (font (size 1.27 1.27)))
     )
-    (property "Footprint" "Connector_PinHeader_2.54mm:PinHeader_2x02_P2.54mm_Vertical_SMD" (at 175.26 215.9 0)
+    (property "Footprint" "Connector_PinHeader_2.54mm:PinHeader_2x02_P2.54mm_Vertical_SMD" (at 175.26 218.44 0)
+      (effects (font (size 1.27 1.27)) hide)
+    )
+    (property "Datasheet" "~" (at 175.26 218.44 0)
+      (effects (font (size 1.27 1.27)) hide)
+    )
+    (property "Manufacturer" "" (at 175.26 218.44 0)
       (effects (font (size 1.27 1.27)) hide)
     )
-    (property "Datasheet" "~" (at 175.26 215.9 0)
+    (property "Mfr. Part No" "" (at 175.26 218.44 0)
+      (effects (font (size 1.27 1.27)) hide)
+    )
+    (property "Description" "" (at 175.26 218.44 0)
       (effects (font (size 1.27 1.27)) hide)
     )
@@
       (effects (font (size 1.27 1.27)) hide)
     )
+    (property "Manufacturer" "" (at 309.88 160.02 0)
+      (effects (font (size 1.27 1.27)) hide)
+    )
+    (property "Mfr. Part No" "" (at 309.88 160.02 0)
+      (effects (font (size 1.27 1.27)) hide)
+    )
+    (property "Description" "" (at 309.88 160.02 0)
+      (effects (font (size 1.27 1.27)) hide)
+    )
     (pin "1")
     (instances
@@
       (effects (font (size 1.27 1.27)) hide)
     )
+    (property "Manufacturer" "" (at 281.94 184.15 0)
+      (effects (font (size 1.27 1.27)) hide)
+    )
+    (property "Mfr. Part No" "" (at 281.94 184.15 0)
+      (effects (font (size 1.27 1.27)) hide)
+    )
+    (property "Description" "" (at 281.94 184.15 0)
+      (effects (font (size 1.27 1.27)) hide)
+    )
     (pin "1")
     (instances
@@
       (effects (font (size 1.27 1.27)) hide)
     )
+    (property "Manufacturer" "" (at 271.78 45.72 0)
+      (effects (font (size 1.27 1.27)) hide)
+    )
+    (property "Mfr. Part No" "" (at 271.78 45.72 0)
+      (effects (font (size 1.27 1.27)) hide)
+    )
+    (property "Description" "" (at 271.78 45.72 0)
+      (effects (font (size 1.27 1.27)) hide)
+    )
     (pin "1")
     (instances
@@
       (effects (font (size 1.27 1.27)) hide)
     )
+    (property "Manufacturer" "" (at 309.88 182.88 0)
+      (effects (font (size 1.27 1.27)) hide)
+    )
+    (property "Mfr. Part No" "" (at 309.88 182.88 0)
+      (effects (font (size 1.27 1.27)) hide)
+    )
+    (property "Description" "" (at 309.88 182.88 0)
+      (effects (font (size 1.27 1.27)) hide)
+    )
     (pin "1")
     (instances
@@
       (effects (font (size 1.27 1.27)) hide)
     )
+    (property "Manufacturer" "" (at 271.78 137.16 0)
+      (effects (font (size 1.27 1.27)) hide)
+    )
+    (property "Mfr. Part No" "" (at 271.78 137.16 0)
+      (effects (font (size 1.27 1.27)) hide)
+    )
+    (property "Description" "" (at 271.78 137.16 0)
+      (effects (font (size 1.27 1.27)) hide)
+    )
     (pin "1")
     (instances
@@
     )
   )
-  (symbol (lib_id "power:VAA") (at 193.04 215.9 0) (unit 1)
+  (symbol (lib_id "power:VAA") (at 194.31 215.9 0) (unit 1)
     (in_bom yes) (on_board yes) (dnp no) (fields_autoplaced)
-    (property "Reference" "#PWR017" (at 193.04 219.71 0)
+    (property "Reference" "#PWR017" (at 194.31 219.71 0)
       (effects (font (size 1.27 1.27)) hide)
     )
-    (property "Value" "VAA" (at 193.04 212.09 0)
+    (property "Value" "VAA" (at 194.31 212.09 0)
       (effects (font (size 1.27 1.27)))
     )
-    (property "Footprint" "" (at 193.04 215.9 0)
+    (property "Footprint" "" (at 194.31 215.9 0)
       (effects (font (size 1.27 1.27)) hide)
     )
-    (property "Datasheet" "" (at 193.04 215.9 0)
+    (property "Datasheet" "" (at 194.31 215.9 0)
       (effects (font (size 1.27 1.27)) hide)
     )

Commit message: routing mostly complete
Parts:
- R86, R88: footprint Resistor_SMD:R_0603_1608Metric -> Resistor_SMD:R_0402_1005Metric
- TP3, TP4: footprint TestPoint:TestPoint_Keystone_5000-5004_Miniature -> SierraLobo:TestPoint_Keystone_5000-5004_Miniature
Connections:
- net LED_PWR renamed LED_VCC
Changed lines of the file:
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@@
     (effects (font (size 1.27 1.27)) (justify right bottom))
   )
-  (global_label "LED_PWR" (shape input) (at 358.14 137.16 180) (fields_autoplaced)
-    (effects (font (size 1.016 1.016)) (justify right))
-    (property "Intersheetrefs" "${INTERSHEET_REFS}" (at 349.6138 137.16 0)
-      (effects (font (size 1.016 1.016)) (justify right) hide)
+  (global_label "LED_VCC" (shape input) (at 358.14 179.07 180) (fields_autoplaced)
+    (effects (font (size 1.27 1.27)) (justify right))
+    (property "Intersheetrefs" "${INTERSHEET_REFS}" (at 347.8451 179.07 0)
+      (effects (font (size 1.27 1.27)) (justify right) hide)
     )
   )
-  (global_label "LED_PWR" (shape input) (at 358.14 179.07 180) (fields_autoplaced)
-    (effects (font (size 1.016 1.016)) (justify right))
-    (property "Intersheetrefs" "${INTERSHEET_REFS}" (at 349.6138 179.07 0)
-      (effects (font (size 1.016 1.016)) (justify right) hide)
+  (global_label "LED_VCC" (shape input) (at 358.14 137.16 180) (fields_autoplaced)
+    (effects (font (size 1.27 1.27)) (justify right))
+    (property "Intersheetrefs" "${INTERSHEET_REFS}" (at 347.8451 137.16 0)
+      (effects (font (size 1.27 1.27)) (justify right) hide)
     )
   )
@@
       (effects (font (size 1.27 1.27)) (justify left) hide)
     )
-    (property "Footprint" "TestPoint:TestPoint_Keystone_5000-5004_Miniature" (at 327.66 190.5 0)
+    (property "Footprint" "SierraLobo:TestPoint_Keystone_5000-5004_Miniature" (at 327.66 190.5 0)
       (effects (font (size 1.27 1.27)) hide)
     )
@@
       (effects (font (size 1.27 1.27)) (justify left) hide)
     )
-    (property "Footprint" "TestPoint:TestPoint_Keystone_5000-5004_Miniature" (at 327.66 167.64 0)
+    (property "Footprint" "SierraLobo:TestPoint_Keystone_5000-5004_Miniature" (at 327.66 167.64 0)
       (effects (font (size 1.27 1.27)) hide)
     )
@@
       (effects (font (size 1.27 1.27)) (justify left) hide)
     )
-    (property "Footprint" "TestPoint:TestPoint_Keystone_5000-5004_Miniature" (at 327.66 182.88 0)
+    (property "Footprint" "SierraLobo:TestPoint_Keystone_5000-5004_Miniature" (at 327.66 182.88 0)
       (effects (font (size 1.27 1.27)) hide)
     )
@@
       (effects (font (size 1.27 1.27)))
     )
-    (property "Footprint" "Resistor_SMD:R_0603_1608Metric" (at 363.474 136.144 90)
+    (property "Footprint" "Resistor_SMD:R_0402_1005Metric" (at 363.474 136.144 90)
       (effects (font (size 1.27 1.27)) hide)
     )
@@
       (effects (font (size 1.27 1.27)) (justify left) hide)
     )
-    (property "Footprint" "TestPoint:TestPoint_Keystone_5000-5004_Miniature" (at 327.66 160.02 0)
+    (property "Footprint" "SierraLobo:TestPoint_Keystone_5000-5004_Miniature" (at 327.66 160.02 0)
       (effects (font (size 1.27 1.27)) hide)
     )
@@
       (effects (font (size 1.27 1.27)))
     )
-    (property "Footprint" "Resistor_SMD:R_0603_1608Metric" (at 363.474 178.054 90)
+    (property "Footprint" "Resistor_SMD:R_0402_1005Metric" (at 363.474 178.054 90)
       (effects (font (size 1.27 1.27)) hide)
     )
@@
       (effects (font (size 1.27 1.27)) (justify left) hide)
     )
-    (property "Footprint" "TestPoint:TestPoint_Keystone_5000-5004_Miniature" (at 327.66 152.4 0)
+    (property "Footprint" "SierraLobo:TestPoint_Keystone_5000-5004_Miniature" (at 327.66 152.4 0)
       (effects (font (size 1.27 1.27)) hide)
     )
@@
       (effects (font (size 1.27 1.27)) (justify left) hide)
     )
-    (property "Footprint" "TestPoint:TestPoint_Keystone_5000-5004_Miniature" (at 327.66 175.26 0)
+    (property "Footprint" "SierraLobo:TestPoint_Keystone_5000-5004_Miniature" (at 327.66 175.26 0)
       (effects (font (size 1.27 1.27)) hide)
     )

Commit message: working
Parts:
- removed J9: Conn_02x02_Top_Bottom, Connector_PinHeader_2.54mm:PinHeader_2x02_P2.54mm_Vertical_SMD, symbol Connector_Generic:Conn_02x02_Odd_Even
- added D4 (x2): 1N4148W-13-F, Diode_SMD:D_SOD-123, symbol Device:D
- added P4: Conn_02x03_Odd_Even, Connector_PinHeader_2.54mm:PinHeader_2x03_P2.54mm_Vertical_SMD, symbol Connector_Generic:Conn_02x03_Odd_Even
- renumbered C61 to C70, C64 to C74, Q4 to Q5, Q6 to Q7, Q9 to Q8, Q3 to Q9, R77 to R82, R85 to R83, R70 to R84, R75 to R85, R80 to R86, R86 to R87, R68 to R88, R76 to R89, R87 to R90, R88 to R91
Connections:
- net 5V_USB: now also C74.1, C8.1, R3.1, U25.1 (OUT), D4.2 (A), P4.3 (Pin_3); no longer C25.1, C8.1, U25.5 (IN)
- net LED_VCC: now also P4.2 (Pin_2), P4.4 (Pin_4), P4.6 (Pin_6)
- net VAA: now also D4.1 (K), D4.1 (K)
- new net 5V_DEBUG: D4.2 (A), P4.1 (Pin_1)
- new net 5V_USB_IN: C25.1, C8.1, U25.5 (IN)
- new net BUS_LED_PWR: P4.5 (Pin_5)
Other:
- note added: "DEBUG LEDs"
- note added: "Debug/Programming Power OR's"
- note added: "GREEN = VAA ORANGE = 3V3D"
- note added: "INPUT BULK CAPS"
- note added: "LED_VCC SELECT HEADER"
- note added: "Protects USB host"
- note added: "USB or 5V_DEBUG may be applied for programming/debug w/o VBATT 5V_A won't work when these are applied (LDO dropout) not reccomended to operate adj. bucks with this low power as well."
- note added: "controlling device can disable power redundant PMOS"
- note added: "controlling device can hard-reset via toggling EN, device can hard-reset itself with this circuitry"
- note added: "led power options for different configurations"
- note removed: "BULK"
- note removed: "JUMPERS"
- title: (none) -> SCHEMATIC, CUBESAT MAGNETORQER DRIVER
- moved on the sheet: C10, C11, C13, C14, C15, C16, C17, C5, C7, C70, C9, LED3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

Commit message: worked review changes
Parts:
- C13: renamed from C70; Manufacturer (none) -> TDK Corporation; Mfr. Part No (none) -> CGA4J1X7S1E106K125AE; Value2 (none) -> 25V
- C16: renamed from C74; Value2 (none) -> 25V
- C? (x3): renamed from C8; Manufacturer (none) -> TDK Corporation; Mfr. Part No (none) -> CGA3E2X7R1H104K080AE; Value2 (none) -> 50V
- C?: renamed from C11; Manufacturer (none) -> TDK Corporation; Mfr. Part No (none) -> CGA4J3X7R1H105K125AE; Value2 (none) -> 50V
- C?: renamed from C16; Manufacturer (none) -> TDK Corporation; Mfr. Part No (none) -> CGA4J3X7R1H105K125AE; Value2 (none) -> 50V
- C?: renamed from C5; Manufacturer (none) -> Vishay Sprague; Value2 (none) -> 16V
- C?: renamed from C7; Manufacturer (none) -> Vishay Sprague; Value2 (none) -> 16V
- C?: renamed from C15; Manufacturer (none) -> TDK Corporation; Mfr. Part No (none) -> CGA4J3X7R1H105K125AE; Value2 (none) -> 50V
- C?: renamed from C17; Manufacturer (none) -> TDK Corporation; Mfr. Part No (none) -> CGA4J1X7S1E106K125AE; Value2 (none) -> 25V
- C?: renamed from C14; Manufacturer (none) -> TDK Corporation; Mfr. Part No (none) -> CGA4J3X7R1H105K125AE; Value2 (none) -> 50V
- C?: renamed from C25; Manufacturer (none) -> TDK Corporation; Mfr. Part No (none) -> CGA4J1X7S1E106K125AE; Value2 (none) -> 25V
- C?: renamed from C13; Manufacturer (none) -> TDK Corporation; Mfr. Part No (none) -> CGA4J3X7R1H105K125AE; Value2 (none) -> 50V
- C?: renamed from C9; Manufacturer (none) -> TDK Corporation; Mfr. Part No (none) -> CGA4J3X7R1H105K125AE; Value2 (none) -> 50V
- C?: renamed from C10; Manufacturer (none) -> TDK Corporation; Mfr. Part No (none) -> CGA4J3X7R1H105K125AE; Value2 (none) -> 50V
- D? (x2): renamed from D4; Value2 (none) -> 100V
- P3: renamed from P4; Manufacturer (none) -> Samtec; Mfr. Part No (none) -> TSM-118-01-T-DV
- Q1: renamed from Q9; Manufacturer (none) -> Diodes Incorporated; Mfr. Part No (none) -> MMDT2222A-7-F
- Q4: renamed from Q7; Manufacturer (none) -> Diodes Incorporated; Mfr. Part No (none) -> MMDT2222A-7-F
- Q7: renamed from Q8; Manufacturer (none) -> Diodes Incorporated; Mfr. Part No (none) -> MMDT2222A-7-F
- Q?: renamed from Q1; Manufacturer (none) -> onsemi; Mfr. Part No (none) -> MMBT4401WT1G
- R13: renamed from R88; Manufacturer (none) -> Stackpole Electronics Inc; Mfr. Part No (none) -> RMCF0603FT10K0; Value2 (none) -> 100mW
- R15: renamed from R84; Manufacturer (none) -> Stackpole Electronics Inc; Mfr. Part No (none) -> RMCF0603FT100K; Value2 (none) -> 100mW
- R20: renamed from R85; Manufacturer (none) -> Stackpole Electronics Inc; Mfr. Part No (none) -> RMCF0603FT200K; Value2 (none) -> 100mW
- R21: renamed from R89; Manufacturer (none) -> Stackpole Electronics Inc; Mfr. Part No (none) -> RMCF0603FT20K0; Value2 (none) -> 100mW
- R22: renamed from R82; Manufacturer (none) -> Stackpole Electronics Inc; Mfr. Part No (none) -> RMCF0603FT100K; Value2 (none) -> 100mW
- R25: renamed from R86; Manufacturer (none) -> Stackpole Electronics Inc; Mfr. Part No (none) -> RMCF0603FT73K2; Value2 (none) -> 100mW
- R30: renamed from R83; Manufacturer (none) -> Stackpole Electronics Inc; Mfr. Part No (none) -> RMCF0402FT1K50; Value2 (none) -> 62.5mW
- R31: renamed from R87; Manufacturer (none) -> Stackpole Electronics Inc; Mfr. Part No (none) -> RMCF0402FT10K0; Value2 (none) -> 62.5mW
- R32: renamed from R90; Manufacturer (none) -> Stackpole Electronics Inc; Mfr. Part No (none) -> RMCF0402FT1K50; Value2 (none) -> 62.5mW
- R33: renamed from R91; Manufacturer (none) -> Stackpole Electronics Inc; Mfr. Part No (none) -> RMCF0402FT10K0; Value2 (none) -> 62.5mW
- R? (x2): renamed from R5; Manufacturer (none) -> Stackpole Electronics Inc; Mfr. Part No (none) -> RMCF0603FG1K00; Value2 (none) -> 100mW
- R? (x2): renamed from R3; Manufacturer (none) -> Stackpole Electronics Inc; Mfr. Part No (none) -> RMCF0603FT10K0; Value2 (none) -> 100mW
- R?: renamed from R8; Manufacturer (none) -> Stackpole Electronics Inc; Mfr. Part No (none) -> RMCF0603FT10K0; Value2 (none) -> 100mW
- R? (x2): renamed from R2; Manufacturer (none) -> Stackpole Electronics Inc; Mfr. Part No (none) -> RMCF0603FT100K; Value2 (none) -> 100mW
- R?: renamed from R9; Manufacturer (none) -> Stackpole Electronics Inc; Mfr. Part No (none) -> RMCF0603FT12K4; Value2 (none) -> 100mW
- R?: renamed from R3; Manufacturer (none) -> Stackpole Electronics Inc; Mfr. Part No (none) -> RMCF0603FT100K; Value2 (none) -> 100mW
- R?: renamed from R2; Manufacturer (none) -> Stackpole Electronics Inc; Mfr. Part No (none) -> RMCF0603FG1K00; Value2 (none) -> 100mW
- R?: renamed from R10; value 4.1k -> 4.12k; Manufacturer (none) -> Stackpole Electronics Inc; Mfr. Part No (none) -> RMCF0603FT4K12; Value2 (none) -> 100mW
- U?: renamed from U6; value ATL431BQ -> ATL431; symbol SierraLobo:TLVH431BQxDBV -> SierraLobo:ATL31BQDBZR; Manufacturer (none) -> Texas Instruments; Mfr. Part No (none) -> ATL431BQDBZR
- renumbered LED3 to LED1, LED4 to LED2, Q5 to Q2, Q3 to Q?, TP4 to TP?, TP3 to TP?, U4 to U?, U25 to U?, U3 to U?, U5 to U?
Other:
- note added: "pull to vin"
